File: hardware/friendship/friendship_v0/frienship_1.sch (EAGLE design)
At the start: 29 parts, among them IC5 741G66DBV, IC6 741G66DBV, IC7 741G66DBV, IC8 741G66DBV

Commit message: fixed wrong routing for differential bus pairs
Parts:
- added R11, R13: 120, rcl:R-EU_R0603
Connections:
- net FASTCLK+: now also R11.1, R13.1
- net FASTCLK-: now also R11.2, R13.2
- net RX+: now also PORT0.BUS1+, PORT1.BUS1+, PORT2.BUS1+, PORT3.BUS1+; no longer PORT0.RX+, PORT1.RX+, PORT2.RX+, PORT3.RX+
- net RX-: now also PORT0.BUS1-, PORT1.BUS1-, PORT2.BUS1-, PORT3.BUS1-; no longer PORT0.RX-, PORT1.RX-, PORT2.RX-, PORT3.RX-
- net TX+: now also PORT0.BUS0+, PORT1.BUS0+, PORT2.BUS0+, PORT3.BUS0+; no longer PORT0.TX+, PORT1.TX+, PORT2.TX+, PORT3.TX+
- net TX-: now also PORT0.BUS0-, PORT1.BUS0-, PORT2.BUS0-, PORT3.BUS0-; no longer PORT0.TX-, PORT1.TX-, PORT2.TX-, PORT3.TX-
Other:
- moved on the sheet: R10, R6, R8, R9
Changed lines of the file:
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@@
 <part name="R9" library="rcl" deviceset="R-EU_" device="R0603" value="120"/>
 <part name="R10" library="rcl" deviceset="R-EU_" device="R0603" value="120"/>
+<part name="R11" library="rcl" deviceset="R-EU_" device="R0603" value="120"/>
+<part name="R13" library="rcl" deviceset="R-EU_" device="R0603" value="120"/>
 </parts>
 <sheets>
@@
 <instance part="GND23" gate="1" x="-146.05" y="173.99"/>
 <instance part="GND29" gate="1" x="-138.43" y="173.99"/>
-<instance part="R6" gate="G$1" x="-22.86" y="250.19" rot="R180"/>
-<instance part="R8" gate="G$1" x="-22.86" y="238.76" rot="R180"/>
-<instance part="R9" gate="G$1" x="-22.86" y="255.27" rot="R180"/>
-<instance part="R10" gate="G$1" x="-22.86" y="243.84" rot="R180"/>
+<instance part="R6" gate="G$1" x="-26.67" y="247.65" rot="R90"/>
+<instance part="R8" gate="G$1" x="-26.67" y="233.68" rot="R90"/>
+<instance part="R9" gate="G$1" x="-21.59" y="247.65" rot="R90"/>
+<instance part="R10" gate="G$1" x="-21.59" y="233.68" rot="R90"/>
+<instance part="R11" gate="G$1" x="-71.12" y="241.3" rot="R270"/>
+<instance part="R13" gate="G$1" x="-77.47" y="241.3" rot="R270"/>
 </instances>
 <busses>
@@
 <bus name="GND,MOSI,CLK,/CS,PPS,FASTCLK+,FASTCLK-,FASTCLK3V3">
 <segment>
-<wire x1="-59.69" y1="-260.35" x2="-59.69" y2="210.82" width="0.762" layer="92"/>
+<wire x1="-59.69" y1="-260.35" x2="-59.69" y2="251.46" width="0.762" layer="92"/>
 </segment>
 </bus>
@@
 <net name="TX-" class="0">
 <segment>
-<pinref part="PORT0" gate="G$1" pin="TX-"/>
+<pinref part="PORT0" gate="G$1" pin="BUS0-"/>
 <wire x1="15.24" y1="134.62" x2="-41.91" y2="134.62" width="0.1524" layer="91"/>
 </segment>
 <segment>
-<pinref part="PORT1" gate="G$1" pin="TX-"/>
+<pinref part="PORT1" gate="G$1" pin="BUS0-"/>
 <wire x1="15.24" y1="19.05" x2="-41.91" y2="19.05" width="0.1524" layer="91"/>
 </segment>
 <segment>
-<pinref part="PORT2" gate="G$1" pin="TX-"/>
+<pinref part="PORT2" gate="G$1" pin="BUS0-"/>
 <wire x1="15.24" y1="-96.52" x2="-41.91" y2="-96.52" width="0.1524" layer="91"/>
 </segment>
 <segment>
-<pinref part="PORT3" gate="G$1" pin="TX-"/>
+<pinref part="PORT3" gate="G$1" pin="BUS0-"/>
 <wire x1="15.24" y1="-210.82" x2="-41.91" y2="-210.82" width="0.1524" layer="91"/>
 </segment>
 <segment>
-<wire x1="-41.91" y1="247.65" x2="-13.97" y2="247.65" width="0.1524" layer="91"/>
-<wire x1="-13.97" y1="247.65" x2="-13.97" y2="250.19" width="0.1524" layer="91"/>
+<pinref part="R9" gate="G$1" pin="1"/>
 <pinref part="R6" gate="G$1" pin="1"/>
-<wire x1="-13.97" y1="250.19" x2="-17.78" y2="250.19" width="0.1524" layer="91"/>
-<wire x1="-13.97" y1="250.19" x2="-13.97" y2="255.27" width="0.1524" layer="91"/>
-<junction x="-13.97" y="250.19"/>
-<pinref part="R9" gate="G$1" pin="1"/>
-<wire x1="-13.97" y1="255.27" x2="-17.78" y2="255.27" width="0.1524" layer="91"/>
+<wire x1="-26.67" y1="242.57" x2="-21.59" y2="242.57" width="0.1524" layer="91"/>
+<junction x="-26.67" y="242.57"/>
+<wire x1="-30.48" y1="245.11" x2="-26.67" y2="242.57" width="0.1524" layer="91"/>
+<wire x1="-41.91" y1="245.11" x2="-30.48" y2="245.11" width="0.1524" layer="91"/>
 </segment>
 </net>
 <net name="TX+" class="0">
 <segment>
-<pinref part="PORT0" gate="G$1" pin="TX+"/>
+<pinref part="PORT0" gate="G$1" pin="BUS0+"/>
 <wire x1="15.24" y1="132.08" x2="-41.91" y2="132.08" width="0.1524" layer="91"/>
 <wire x1="-41.91" y1="132.08" x2="-41.91" y2="130.81" width="0.1524" layer="91"/>
 </segment>
 <segment>
-<pinref part="PORT1" gate="G$1" pin="TX+"/>
+<pinref part="PORT1" gate="G$1" pin="BUS0+"/>
 <wire x1="15.24" y1="16.51" x2="-41.91" y2="16.51" width="0.1524" layer="91"/>
 </segment>
 <segment>
-<pinref part="PORT2" gate="G$1" pin="TX+"/>
+<pinref part="PORT2" gate="G$1" pin="BUS0+"/>
 <wire x1="15.24" y1="-99.06" x2="-41.91" y2="-99.06" width="0.1524" layer="91"/>
 </segment>
 <segment>
-<pinref part="PORT3" gate="G$1" pin="TX+"/>
+<pinref part="PORT3" gate="G$1" pin="BUS0+"/>
 <wire x1="15.24" y1="-213.36" x2="-41.91" y2="-213.36" width="0.1524" layer="91"/>
 </segment>
@@
 <wire x1="-41.91" y1="250.19" x2="-30.48" y2="250.19" width="0.1524" layer="91"/>
 <pinref part="R6" gate="G$1" pin="2"/>
-<wire x1="-30.48" y1="250.19" x2="-27.94" y2="250.19" width="0.1524" layer="91"/>
+<wire x1="-30.48" y1="250.19" x2="-26.67" y2="252.73" width="0.1524" layer="91"/>
 <pinref part="R9" gate="G$1" pin="2"/>
-<wire x1="-30.48" y1="250.19" x2="-30.48" y2="255.27" width="0.1524" layer="91"/>
-<wire x1="-30.48" y1="255.27" x2="-27.94" y2="255.27" width="0.1524" layer="91"/>
-<junction x="-30.48" y="250.19"/>
+<wire x1="-26.67" y1="252.73" x2="-21.59" y2="252.73" width="0.1524" layer="91"/>
+<junction x="-26.67" y="252.73"/>
 </segment>
 </net>
@@
 <net name="RX+" class="0">
 <segment>
-<pinref part="PORT0" gate="G$1" pin="RX+"/>
+<pinref part="PORT0" gate="G$1" pin="BUS1+"/>
 <wire x1="15.24" y1="127" x2="-41.91" y2="127" width="0.1524" layer="91"/>
 </segment>
 <segment>
-<pinref part="PORT1" gate="G$1" pin="RX+"/>
+<pinref part="PORT1" gate="G$1" pin="BUS1+"/>
 <wire x1="15.24" y1="11.43" x2="-41.91" y2="11.43" width="0.1524" layer="91"/>
 </segment>
 <segment>
-<pinref part="PORT2" gate="G$1" pin="RX+"/>
+<pinref part="PORT2" gate="G$1" pin="BUS1+"/>
 <wire x1="15.24" y1="-104.14" x2="-41.91" y2="-104.14" width="0.1524" layer="91"/>
 </segment>
 <segment>
-<pinref part="PORT3" gate="G$1" pin="RX+"/>
+<pinref part="PORT3" gate="G$1" pin="BUS1+"/>
 <wire x1="15.24" y1="-218.44" x2="-41.91" y2="-218.44" width="0.1524" layer="91"/>
 </segment>
 <segment>
 <pinref part="R8" gate="G$1" pin="2"/>
-<wire x1="-41.91" y1="238.76" x2="-30.48" y2="238.76" width="0.1524" layer="91"/>
+<wire x1="-41.91" y1="236.22" x2="-30.48" y2="236.22" width="0.1524" layer="91"/>
+<wire x1="-30.48" y1="236.22" x2="-26.67" y2="238.76" width="0.1524" layer="91"/>
 <pinref part="R10" gate="G$1" pin="2"/>
-<wire x1="-30.48" y1="238.76" x2="-27.94" y2="238.76" width="0.1524" layer="91"/>
-<wire x1="-30.48" y1="238.76" x2="-30.48" y2="243.84" width="0.1524" layer="91"/>
-<wire x1="-30.48" y1="243.84" x2="-27.94" y2="243.84" width="0.1524" layer="91"/>
-<junction x="-30.48" y="238.76"/>
+<wire x1="-26.67" y1="238.76" x2="-21.59" y2="238.76" width="0.1524" layer="91"/>
+<junction x="-26.67" y="238.76"/>
 </segment>
 </net>
@@
 <segment>
 <wire x1="15.24" y1="124.46" x2="-41.91" y2="124.46" width="0.1524" layer="91"/>
-<pinref part="PORT0" gate="G$1" pin="RX-"/>
-</segment>
-<segment>
-<pinref part="PORT1" gate="G$1" pin="RX-"/>
+<pinref part="PORT0" gate="G$1" pin="BUS1-"/>
+</segment>
+<segment>
+<pinref part="PORT1" gate="G$1" pin="BUS1-"/>
 <wire x1="15.24" y1="8.89" x2="-41.91" y2="8.89" width="0.1524" layer="91"/>
 </segment>
 <segment>
-<pinref part="PORT2" gate="G$1" pin="RX-"/>
+<pinref part="PORT2" gate="G$1" pin="BUS1-"/>
 <wire x1="15.24" y1="-106.68" x2="-41.91" y2="-106.68" width="0.1524" layer="91"/>
 </segment>
 <segment>
-<pinref part="PORT3" gate="G$1" pin="RX-"/>
+<pinref part="PORT3" gate="G$1" pin="BUS1-"/>
 <wire x1="15.24" y1="-220.98" x2="-41.91" y2="-220.98" width="0.1524" layer="91"/>
 </segment>
 <segment>
-<wire x1="-41.91" y1="236.22" x2="-13.97" y2="236.22" width="0.1524" layer="91"/>
-<wire x1="-13.97" y1="236.22" x2="-13.97" y2="238.76" width="0.1524" layer="91"/>
+<wire x1="-41.91" y1="231.14" x2="-30.48" y2="231.14" width="0.1524" layer="91"/>
+<wire x1="-30.48" y1="231.14" x2="-26.67" y2="228.6" width="0.1524" layer="91"/>
 <pinref part="R8" gate="G$1" pin="1"/>
-<wire x1="-13.97" y1="238.76" x2="-17.78" y2="238.76" width="0.1524" layer="91"/>
+<wire x1="-21.59" y1="228.6" x2="-26.67" y2="228.6" width="0.1524" layer="91"/>
 <pinref part="R10" gate="G$1" pin="1"/>
-<wire x1="-13.97" y1="238.76" x2="-13.97" y2="243.84" width="0.1524" layer="91"/>
-<wire x1="-13.97" y1="243.84" x2="-17.78" y2="243.84" width="0.1524" layer="91"/>
-<junction x="-13.97" y="238.76"/>
+<junction x="-21.59" y="228.6"/>
 </segment>
 </net>
@@
 <wire x1="15.24" y1="-243.84" x2="-59.69" y2="-243.84" width="0.1524" layer="91"/>
 </segment>
+<segment>
+<pinref part="R11" gate="G$1" pin="1"/>
+<wire x1="-59.69" y1="247.65" x2="-71.12" y2="247.65" width="0.1524" layer="91"/>
+<wire x1="-71.12" y1="247.65" x2="-71.12" y2="246.38" width="0.1524" layer="91"/>
+<pinref part="R13" gate="G$1" pin="1"/>
+<wire x1="-77.47" y1="246.38" x2="-77.47" y2="247.65" width="0.1524" layer="91"/>
+<wire x1="-77.47" y1="247.65" x2="-71.12" y2="247.65" width="0.1524" layer="91"/>
+<junction x="-71.12" y="247.65"/>
+</segment>
 </net>
 <net name="FASTCLK-" class="0">
@@
 <wire x1="15.24" y1="-246.38" x2="-59.69" y2="-246.38" width="0.1524" layer="91"/>
 </segment>
-</net>
+<segment>
+<wire x1="-59.69" y1="234.95" x2="-71.12" y2="234.95" width="0.1524" layer="91"/>
+<pinref part="R11" gate="G$1" pin="2"/>
+<wire x1="-71.12" y1="234.95" x2="-71.12" y2="236.22" width="0.1524" layer="91"/>
+<pinref part="R13" gate="G$1" pin="2"/>
+<wire x1="-77.47" y1="236.22" x2="-77.47" y2="234.95" width="0.1524" layer="91"/>
+<wire x1="-77.47" y1="234.95" x2="-71.12" y2="234.95" width="0.1524" layer="91"/>
+<junction x="-71.12" y="234.95"/>
+</segment>
+</net>
