File: hardware/flutter/eagle/FPGA_Board.sch (EAGLE design)
At the start: 60 parts, among them IC1 AT45DB161D-SU, IC2 MEGA8-AI, IC3 MAX3468CSA, Q1 8Mhz, U2 XC3S50AVQ100

Commit message: changed level converter for rs48 from max488 to max481 (similar to max485)
Parts:
- IC3: value MAX3468CSA -> MAX481CSA; device maxim:MAX3468CSA -> maxim:MAX481CSA
Connections:
- removed net UC_RX+: IC3.DI, U$4.TX+
- removed net UC_RX-: IC3.DE, U$4.TX-
- removed net UC_TX+: IC3.RO, U$4.RX+
- removed net UC_TX-: IC3.RE/, U$4.RX-
- new net BUS0+: IC3G$1.A, U$4.BUS0+
- new net BUS0-: IC3G$1.B, U$4.BUS0-
- new net BUS1+: U$4.BUS1+
- new net BUS1-: U$4.BUS1-
- net +5V: now also IC3P.VCC
- net GND: now also IC3P.GND; no longer IC3.GND
- net N$10: now also IC3G$1.RO; no longer IC3.A
- net N$5: now also IC2.PD2(INT0), IC3G$1.DE, IC3G$1.RE/; no longer IC3.VCC
- net N$6: now also IC3G$1.DI; no longer IC3.B
Changed lines of the file:
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@@
 <part name="GND24" library="supply1" deviceset="GND" device=""/>
 <part name="JP3" library="pinhead" deviceset="PINHD-2X5" device="" value="ISP"/>
-<part name="IC3" library="maxim" deviceset="MAX34*" device="SA" technology="68C"/>
 <part name="P+8" library="supply1" deviceset="+5V" device=""/>
 <part name="GND25" library="supply1" deviceset="GND" device=""/>
@@
 <part name="P+9" library="supply1" deviceset="+5V" device=""/>
 <part name="U$5" library="hgg" deviceset="HGG_LOGO" device=""/>
+<part name="IC3" library="maxim" deviceset="MAX481CSA" device=""/>
 </parts>
 <sheets>
@@
 <instance part="GND24" gate="1" x="337.82" y="172.72" rot="R270"/>
 <instance part="JP3" gate="A" x="497.84" y="149.86"/>
-<instance part="IC3" gate="G$1" x="485.14" y="185.42" rot="R180"/>
-<instance part="P+8" gate="1" x="449.58" y="177.8"/>
-<instance part="GND25" gate="1" x="457.2" y="193.04" rot="R270"/>
+<instance part="P+8" gate="1" x="490.22" y="226.06"/>
+<instance part="GND25" gate="1" x="490.22" y="198.12"/>
 <instance part="GND26" gate="1" x="434.34" y="185.42" rot="R270"/>
 <instance part="R16" gate="G$1" x="457.2" y="185.42"/>
@@
 <instance part="P+9" gate="1" x="269.24" y="99.06"/>
 <instance part="U$5" gate="G$1" x="2.54" y="2.54"/>
+<instance part="IC3" gate="G$1" x="487.68" y="182.88" smashed="yes">
+<attribute name="NAME" x="477.52" y="196.85" size="1.778" layer="95"/>
+<attribute name="VALUE" x="477.52" y="167.64" size="1.778" layer="96"/>
+</instance>
+<instance part="IC3" gate="P" x="490.22" y="210.82"/>
 </instances>
 <busses>
@@
 </segment>
 <segment>
-<pinref part="IC3" gate="G$1" pin="GND"/>
 <pinref part="GND25" gate="1" pin="GND"/>
-<wire x1="464.82" y1="193.04" x2="459.74" y2="193.04" width="0.1524" layer="91"/>
+<wire x1="490.22" y1="203.2" x2="490.22" y2="200.66" width="0.1524" layer="91"/>
+<pinref part="IC3" gate="P" pin="GND"/>
 </segment>
 <segment>
@@
 <segment>
 <pinref part="P+8" gate="1" pin="+5V"/>
-<wire x1="449.58" y1="175.26" x2="449.58" y2="172.72" width="0.1524" layer="91"/>
+<wire x1="490.22" y1="223.52" x2="490.22" y2="218.44" width="0.1524" layer="91"/>
+<pinref part="IC3" gate="P" pin="VCC"/>
 </segment>
 <segment>
@@
 <segment>
 <pinref part="IC2" gate="G$1" pin="PD1(TXD)"/>
-<pinref part="IC3" gate="G$1" pin="B"/>
-<wire x1="426.72" y1="180.34" x2="464.82" y2="180.34" width="0.1524" layer="91"/>
-</segment>
-</net>
-<net name="N$5" class="0">
-<segment>
-<pinref part="IC3" gate="G$1" pin="VCC"/>
-<wire x1="464.82" y1="172.72" x2="449.58" y2="172.72" width="0.1524" layer="91"/>
+<wire x1="426.72" y1="180.34" x2="467.36" y2="180.34" width="0.1524" layer="91"/>
+<wire x1="467.36" y1="180.34" x2="467.36" y2="175.26" width="0.1524" layer="91"/>
+<pinref part="IC3" gate="G$1" pin="DI"/>
+<wire x1="467.36" y1="175.26" x2="474.98" y2="175.26" width="0.1524" layer="91"/>
 </segment>
 </net>
@@
 <segment>
 <pinref part="R16" gate="G$1" pin="2"/>
-<pinref part="IC3" gate="G$1" pin="A"/>
-<wire x1="462.28" y1="185.42" x2="464.82" y2="185.42" width="0.1524" layer="91"/>
-</segment>
-</net>
-<net name="UC_RX+" class="0">
-<segment>
-<pinref part="IC3" gate="G$1" pin="DI"/>
-<wire x1="497.84" y1="190.5" x2="523.24" y2="190.5" width="0.1524" layer="91"/>
-<label x="518.16" y="190.5" size="1.778" layer="95"/>
-</segment>
-<segment>
-<pinref part="U$4" gate="G$1" pin="TX+"/>
-<wire x1="172.72" y1="53.34" x2="137.16" y2="53.34" width="0.1524" layer="91"/>
-<label x="137.16" y="53.34" size="1.778" layer="95"/>
-</segment>
-</net>
-<net name="UC_RX-" class="0">
-<segment>
-<pinref part="IC3" gate="G$1" pin="DE"/>
-<wire x1="497.84" y1="185.42" x2="523.24" y2="185.42" width="0.1524" layer="91"/>
-<label x="518.16" y="185.42" size="1.778" layer="95"/>
-</segment>
-<segment>
-<pinref part="U$4" gate="G$1" pin="TX-"/>
-<wire x1="172.72" y1="55.88" x2="137.16" y2="55.88" width="0.1524" layer="91"/>
-<label x="137.16" y="55.88" size="1.778" layer="95"/>
-</segment>
-</net>
-<net name="UC_TX-" class="0">
-<segment>
-<pinref part="IC3" gate="G$1" pin="RE/"/>
-<wire x1="497.84" y1="180.34" x2="523.24" y2="180.34" width="0.1524" layer="91"/>
-<label x="518.16" y="180.34" size="1.778" layer="95"/>
-</segment>
-<segment>
-<pinref part="U$4" gate="G$1" pin="RX-"/>
+<wire x1="462.28" y1="185.42" x2="467.36" y2="185.42" width="0.1524" layer="91"/>
+<wire x1="467.36" y1="185.42" x2="467.36" y2="190.5" width="0.1524" layer="91"/>
+<pinref part="IC3" gate="G$1" pin="RO"/>
+<wire x1="467.36" y1="190.5" x2="474.98" y2="190.5" width="0.1524" layer="91"/>
+</segment>
+</net>
+<net name="BUS1-" class="0">
+<segment>
+<pinref part="U$4" gate="G$1" pin="BUS1-"/>
 <wire x1="172.72" y1="45.72" x2="137.16" y2="45.72" width="0.1524" layer="91"/>
 <label x="137.16" y="45.72" size="1.778" layer="95"/>
 </segment>
 </net>
-<net name="UC_TX+" class="0">
-<segment>
-<pinref part="IC3" gate="G$1" pin="RO"/>
-<wire x1="497.84" y1="175.26" x2="523.24" y2="175.26" width="0.1524" layer="91"/>
-<label x="518.16" y="175.26" size="1.778" layer="95"/>
-</segment>
-<segment>
-<pinref part="U$4" gate="G$1" pin="RX+"/>
+<net name="BUS1+" class="0">
+<segment>
+<pinref part="U$4" gate="G$1" pin="BUS1+"/>
 <wire x1="172.72" y1="48.26" x2="137.16" y2="48.26" width="0.1524" layer="91"/>
 <label x="137.16" y="48.26" size="1.778" layer="95"/>
@@
 </segment>
 </net>
+<net name="N$5" class="0">
+<segment>
+<pinref part="IC3" gate="G$1" pin="RE/"/>
+<pinref part="IC3" gate="G$1" pin="DE"/>
+<wire x1="474.98" y1="185.42" x2="474.98" y2="180.34" width="0.1524" layer="91"/>
+<pinref part="IC2" gate="G$1" pin="PD2(INT0)"/>
+<wire x1="426.72" y1="177.8" x2="474.98" y2="177.8" width="0.1524" layer="91"/>
+<wire x1="474.98" y1="177.8" x2="474.98" y2="180.34" width="0.1524" layer="91"/>
+<junction x="474.98" y="180.34"/>
+</segment>
+</net>
+<net name="BUS0-" class="0">
+<segment>
+<pinref part="IC3" gate="G$1" pin="B"/>
+<wire x1="500.38" y1="185.42" x2="518.16" y2="185.42" width="0.1524" layer="91"/>
+<label x="513.08" y="185.42" size="1.778" layer="95"/>
+</segment>
+<segment>
+<pinref part="U$4" gate="G$1" pin="BUS0-"/>
+<wire x1="172.72" y1="55.88" x2="137.16" y2="55.88" width="0.1524" layer="91"/>
+<label x="137.16" y="55.88" size="1.778" layer="95"/>
+</segment>
+</net>
+<net name="BUS0+" class="0">
+<segment>
+<pinref part="IC3" gate="G$1" pin="A"/>
+<wire x1="500.38" y1="180.34" x2="518.16" y2="180.34" width="0.1524" layer="91"/>
+<label x="513.08" y="180.34" size="1.778" layer="95"/>
+</segment>
+<segment>
+<pinref part="U$4" gate="G$1" pin="BUS0+"/>
+<wire x1="172.72" y1="53.34" x2="137.16" y2="53.34" width="0.1524" layer="91"/>
+<label x="137.16" y="53.34" size="1.778" layer="95"/>
+</segment>
+</net>

Commit message: added GPS module to hgg.lbr and circuit of fpga timing board
Parts:
- added U$6: GPS, hgg:GPS
Changed lines of the file:
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@@
 <part name="U$5" library="hgg" deviceset="HGG_LOGO" device=""/>
 <part name="IC3" library="maxim" deviceset="MAX481CSA" device=""/>
+<part name="U$6" library="hgg" deviceset="GPS" device=""/>
 </parts>
 <sheets>
@@
 <wire x1="0" y1="355.6" x2="0" y2="317.5" width="0.1524" layer="97"/>
 <text x="2.54" y="350.52" size="1.778" layer="97">FPGA_SPI_Clock</text>
+<wire x1="322.58" y1="236.22" x2="322.58" y2="312.42" width="0.1524" layer="97"/>
+<wire x1="419.1" y1="236.22" x2="322.58" y2="236.22" width="0.1524" layer="97"/>
+<wire x1="419.1" y1="312.42" x2="322.58" y2="312.42" width="0.1524" layer="97"/>
+<wire x1="419.1" y1="312.42" x2="419.1" y2="236.22" width="0.1524" layer="97"/>
 </plain>
 <instances>
@@
 </instance>
 <instance part="IC3" gate="P" x="490.22" y="210.82"/>
+<instance part="U$6" gate="G$1" x="368.3" y="274.32"/>
 </instances>
 <busses>
