File: hardware/flutter/eagle/FPGA_Board.sch (EAGLE design)
At the start: 81 parts, among them IC1 AT45DB161D-SU, IC2 MEGA8-AI, IC3 MAX481CSA, Q1 8Mhz, U2 XC3S50AVQ100, X1 BU-SMA-V, X2 MINI-USB-32005-201

Commit message: routes are 20% cooler now
Other:
- note added: "Testpoints"
- moved on the sheet: TP1, TP10, TP11, TP12, TP13, TP14, TP15, TP16, TP17, TP18, TP2, TP3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
Changed lines of the file:
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@@
 <wire x1="444.5" y1="312.42" x2="322.58" y2="312.42" width="0.1524" layer="97"/>
 <wire x1="444.5" y1="312.42" x2="444.5" y2="236.22" width="0.1524" layer="97"/>
+<wire x1="269.24" y1="355.6" x2="124.46" y2="355.6" width="0.1524" layer="97"/>
+<wire x1="269.24" y1="317.5" x2="124.46" y2="317.5" width="0.1524" layer="97"/>
+<wire x1="124.46" y1="355.6" x2="124.46" y2="317.5" width="0.1524" layer="97"/>
+<wire x1="269.24" y1="355.6" x2="269.24" y2="317.5" width="0.1524" layer="97"/>
+<text x="127" y="350.52" size="1.778" layer="97">Testpoints</text>
 </plain>
 <instances>
@@
 <instance part="GND47" gate="1" x="406.4" y="254" rot="R270"/>
 <instance part="X2" gate="G$1" x="429.26" y="281.94"/>
-<instance part="TP1" gate="G$1" x="132.08" y="347.98"/>
-<instance part="TP2" gate="G$1" x="139.7" y="347.98"/>
-<instance part="TP3" gate="G$1" x="147.32" y="347.98"/>
-<instance part="TP4" gate="G$1" x="154.94" y="347.98"/>
-<instance part="TP5" gate="G$1" x="162.56" y="347.98"/>
-<instance part="TP6" gate="G$1" x="170.18" y="347.98"/>
-<instance part="TP7" gate="G$1" x="177.8" y="347.98"/>
-<instance part="TP8" gate="G$1" x="185.42" y="347.98"/>
-<instance part="TP9" gate="G$1" x="193.04" y="347.98"/>
-<instance part="TP10" gate="G$1" x="200.66" y="347.98"/>
-<instance part="TP11" gate="G$1" x="208.28" y="347.98"/>
-<instance part="TP12" gate="G$1" x="215.9" y="347.98"/>
-<instance part="TP13" gate="G$1" x="223.52" y="347.98"/>
-<instance part="TP14" gate="G$1" x="231.14" y="347.98"/>
-<instance part="TP15" gate="G$1" x="238.76" y="347.98"/>
-<instance part="TP16" gate="G$1" x="246.38" y="347.98"/>
-<instance part="TP17" gate="G$1" x="254" y="347.98"/>
-<instance part="TP18" gate="G$1" x="261.62" y="347.98"/>
+<instance part="TP1" gate="G$1" x="132.08" y="345.44"/>
+<instance part="TP2" gate="G$1" x="139.7" y="345.44"/>
+<instance part="TP3" gate="G$1" x="147.32" y="345.44"/>
+<instance part="TP4" gate="G$1" x="154.94" y="345.44"/>
+<instance part="TP5" gate="G$1" x="162.56" y="345.44"/>
+<instance part="TP6" gate="G$1" x="170.18" y="345.44"/>
+<instance part="TP7" gate="G$1" x="177.8" y="345.44"/>
+<instance part="TP8" gate="G$1" x="185.42" y="345.44"/>
+<instance part="TP9" gate="G$1" x="193.04" y="345.44"/>
+<instance part="TP10" gate="G$1" x="200.66" y="345.44"/>
+<instance part="TP11" gate="G$1" x="208.28" y="345.44"/>
+<instance part="TP12" gate="G$1" x="215.9" y="345.44"/>
+<instance part="TP13" gate="G$1" x="223.52" y="345.44"/>
+<instance part="TP14" gate="G$1" x="231.14" y="345.44"/>
+<instance part="TP15" gate="G$1" x="238.76" y="345.44"/>
+<instance part="TP16" gate="G$1" x="246.38" y="345.44"/>
+<instance part="TP17" gate="G$1" x="254" y="345.44"/>
+<instance part="TP18" gate="G$1" x="261.62" y="345.44"/>
 <instance part="JP4" gate="A" x="271.78" y="208.28"/>
 <instance part="GND26" gate="1" x="299.72" y="187.96"/>
@@
 <segment>
 <pinref part="TP1" gate="G$1" pin="TP"/>
-<wire x1="132.08" y1="345.44" x2="132.08" y2="322.58" width="0.1524" layer="91"/>
-<label x="132.08" y="322.58" size="1.778" layer="95" rot="R90"/>
+<wire x1="132.08" y1="342.9" x2="132.08" y2="320.04" width="0.1524" layer="91"/>
+<label x="132.08" y="320.04" size="1.778" layer="95" rot="R90"/>
 </segment>
 </net>
@@
 <segment>
 <pinref part="TP2" gate="G$1" pin="TP"/>
-<wire x1="139.7" y1="345.44" x2="139.7" y2="322.58" width="0.1524" layer="91"/>
-<label x="139.7" y="322.58" size="1.778" layer="95" rot="R90"/>
+<wire x1="139.7" y1="342.9" x2="139.7" y2="320.04" width="0.1524" layer="91"/>
+<label x="139.7" y="320.04" size="1.778" layer="95" rot="R90"/>
 </segment>
 <segment>
@@
 <segment>
 <pinref part="TP3" gate="G$1" pin="TP"/>
-<wire x1="147.32" y1="345.44" x2="147.32" y2="322.58" width="0.1524" layer="91"/>
-<label x="147.32" y="322.58" size="1.778" layer="95" rot="R90"/>
+<wire x1="147.32" y1="342.9" x2="147.32" y2="320.04" width="0.1524" layer="91"/>
+<label x="147.32" y="320.04" size="1.778" layer="95" rot="R90"/>
 </segment>
 </net>
@@
 <segment>
 <pinref part="TP4" gate="G$1" pin="TP"/>
-<wire x1="154.94" y1="345.44" x2="154.94" y2="322.58" width="0.1524" layer="91"/>
-<label x="154.94" y="322.58" size="1.778" layer="95" rot="R90"/>
+<wire x1="154.94" y1="342.9" x2="154.94" y2="320.04" width="0.1524" layer="91"/>
+<label x="154.94" y="320.04" size="1.778" layer="95" rot="R90"/>
 </segment>
 </net>
@@
 <segment>
 <pinref part="TP9" gate="G$1" pin="TP"/>
-<wire x1="193.04" y1="345.44" x2="193.04" y2="322.58" width="0.1524" layer="91"/>
-<label x="193.04" y="322.58" size="1.778" layer="95" rot="R90"/>
+<wire x1="193.04" y1="342.9" x2="193.04" y2="320.04" width="0.1524" layer="91"/>
+<label x="193.04" y="320.04" size="1.778" layer="95" rot="R90"/>
 </segment>
 </net>
@@
 <segment>
 <pinref part="TP15" gate="G$1" pin="TP"/>
-<wire x1="238.76" y1="345.44" x2="238.76" y2="322.58" width="0.1524" layer="91"/>
-<label x="238.76" y="322.58" size="1.778" layer="95" rot="R90"/>
+<wire x1="238.76" y1="342.9" x2="238.76" y2="320.04" width="0.1524" layer="91"/>
+<label x="238.76" y="320.04" size="1.778" layer="95" rot="R90"/>
 </segment>
 </net>
@@
 <segment>
 <pinref part="TP13" gate="G$1" pin="TP"/>
-<wire x1="223.52" y1="345.44" x2="223.52" y2="322.58" width="0.1524" layer="91"/>
-<label x="223.52" y="322.58" size="1.778" layer="95" rot="R90"/>
+<wire x1="223.52" y1="342.9" x2="223.52" y2="320.04" width="0.1524" layer="91"/>
+<label x="223.52" y="320.04" size="1.778" layer="95" rot="R90"/>
 </segment>
 </net>
@@
 <segment>
 <pinref part="TP14" gate="G$1" pin="TP"/>
-<wire x1="231.14" y1="345.44" x2="231.14" y2="322.58" width="0.1524" layer="91"/>
-<label x="231.14" y="322.58" size="1.778" layer="95" rot="R90"/>
+<wire x1="231.14" y1="342.9" x2="231.14" y2="320.04" width="0.1524" layer="91"/>
+<label x="231.14" y="320.04" size="1.778" layer="95" rot="R90"/>
 </segment>
 </net>
@@
 <segment>
 <pinref part="TP5" gate="G$1" pin="TP"/>
-<wire x1="162.56" y1="345.44" x2="162.56" y2="322.58" width="0.1524" layer="91"/>
-<label x="162.56" y="322.58" size="1.778" layer="95" rot="R90"/>
+<wire x1="162.56" y1="342.9" x2="162.56" y2="320.04" width="0.1524" layer="91"/>
+<label x="162.56" y="320.04" size="1.778" layer="95" rot="R90"/>
 </segment>
 </net>
@@
 <segment>
 <pinref part="TP6" gate="G$1" pin="TP"/>
-<wire x1="170.18" y1="345.44" x2="170.18" y2="322.58" width="0.1524" layer="91"/>
-<label x="170.18" y="322.58" size="1.778" layer="95" rot="R90"/>
+<wire x1="170.18" y1="342.9" x2="170.18" y2="320.04" width="0.1524" layer="91"/>
+<label x="170.18" y="320.04" size="1.778" layer="95" rot="R90"/>
 </segment>
 <segment>
@@
 <segment>
 <pinref part="TP7" gate="G$1" pin="TP"/>
-<wire x1="177.8" y1="345.44" x2="177.8" y2="322.58" width="0.1524" layer="91"/>
-<label x="177.8" y="322.58" size="1.778" layer="95" rot="R90"/>
+<wire x1="177.8" y1="342.9" x2="177.8" y2="320.04" width="0.1524" layer="91"/>
+<label x="177.8" y="320.04" size="1.778" layer="95" rot="R90"/>
 </segment>
 </net>
@@
 <segment>
 <pinref part="TP16" gate="G$1" pin="TP"/>
-<wire x1="246.38" y1="345.44" x2="246.38" y2="322.58" width="0.1524" layer="91"/>
-<label x="246.38" y="322.58" size="1.778" layer="95" rot="R90"/>
+<wire x1="246.38" y1="342.9" x2="246.38" y2="320.04" width="0.1524" layer="91"/>
+<label x="246.38" y="320.04" size="1.778" layer="95" rot="R90"/>
 </segment>
 </net>
@@
 <segment>
 <pinref part="TP18" gate="G$1" pin="TP"/>
-<wire x1="261.62" y1="345.44" x2="261.62" y2="322.58" width="0.1524" layer="91"/>
-<label x="261.62" y="322.58" size="1.778" layer="95" rot="R90"/>
+<wire x1="261.62" y1="342.9" x2="261.62" y2="320.04" width="0.1524" layer="91"/>
+<label x="261.62" y="320.04" size="1.778" layer="95" rot="R90"/>
 </segment>
 </net>
@@
 <segment>
 <pinref part="TP17" gate="G$1" pin="TP"/>
-<wire x1="254" y1="345.44" x2="254" y2="322.58" width="0.1524" layer="91"/>
-<label x="254" y="322.58" size="1.778" layer="95" rot="R90"/>
+<wire x1="254" y1="342.9" x2="254" y2="320.04" width="0.1524" layer="91"/>
+<label x="254" y="320.04" size="1.778" layer="95" rot="R90"/>
 </segment>
 </net>
@@
 <segment>
 <pinref part="TP12" gate="G$1" pin="TP"/>
-<wire x1="215.9" y1="345.44" x2="215.9" y2="322.58" width="0.1524" layer="91"/>
-<label x="215.9" y="322.58" size="1.778" layer="95" rot="R90"/>
+<wire x1="215.9" y1="342.9" x2="215.9" y2="320.04" width="0.1524" layer="91"/>
+<label x="215.9" y="320.04" size="1.778" layer="95" rot="R90"/>
 </segment>
 </net>
@@
 <segment>
 <pinref part="TP10" gate="G$1" pin="TP"/>
-<wire x1="200.66" y1="345.44" x2="200.66" y2="322.58" width="0.1524" layer="91"/>
-<label x="200.66" y="322.58" size="1.778" layer="95" rot="R90"/>
+<wire x1="200.66" y1="342.9" x2="200.66" y2="320.04" width="0.1524" layer="91"/>
+<label x="200.66" y="320.04" size="1.778" layer="95" rot="R90"/>
 </segment>
 </net>
@@
 <segment>
 <pinref part="TP11" gate="G$1" pin="TP"/>
-<wire x1="208.28" y1="345.44" x2="208.28" y2="322.58" width="0.1524" layer="91"/>
-<label x="208.28" y="322.58" size="1.778" layer="95" rot="R90"/>
+<wire x1="208.28" y1="342.9" x2="208.28" y2="320.04" width="0.1524" layer="91"/>
+<label x="208.28" y="320.04" size="1.778" layer="95" rot="R90"/>
 </segment>
 </net>
@@
 <segment>
 <pinref part="TP8" gate="G$1" pin="TP"/>
-<wire x1="185.42" y1="345.44" x2="185.42" y2="322.58" width="0.1524" layer="91"/>
-<label x="185.42" y="322.58" size="1.778" layer="95" rot="R90"/>
-</segment>
-</net>
+<wire x1="185.42" y1="342.9" x2="185.42" y2="320.04" width="0.1524" layer="91"/>
+<label x="185.42" y="320.04" size="1.778" layer="95" rot="R90"/>
+</segment>
+</net>
