File: hardware/braeburn/braeburn0/power.sch (EAGLE design)
At the start: 52 parts, among them IC1 7812TV, IC2 7805TV, IC3 7805TV, IC4 ATMEGA48/88/168-AU

Commit message: fixed my fail on use of a zdiode (thanks to samuel), and stuff
Parts:
- added JP1: (no value), jumper:JP1E
- added R6: (no value), resistor:R-EU_R0805
- renumbered R5 to 0OHM
Connections:
- new net N$27: C19.1, C20.1, IC4.VCC@1, IC4.VCC@2, JP1.1, L7.2, R6.1, SV1.2
- net GND: now also D5.A
- net N$14: now also IC4.PC6(/RESET/PCINT14), R6.2, SV1.5; no longer C11.1, D5.A, L3.1
- net N$4: now also C11.1, L3.1
- net N$9: now also JP1.2; no longer C19.1, C20.1, IC4.PC6(/RESET/PCINT14), IC4.VCC@1, IC4.VCC@2, L7.2, SV1.2, SV1.5
Other:
- moved on the sheet: D5
Changed lines of the file:
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@@
 <part name="C20" library="rcl" deviceset="C-EU" device="C0805"/>
 <part name="GND28" library="supply1" deviceset="GND" device=""/>
-<part name="R5" library="rcl" deviceset="R-EU_" device="0411/15"/>
+<part name="0OHM" library="rcl" deviceset="R-EU_" device="0411/15"/>
 <part name="L8" library="rcl" deviceset="L-EU" device="0207/5V"/>
 <part name="L9" library="rcl" deviceset="L-EU" device="0207/5V"/>
@@
 <part name="C21" library="rcl" deviceset="C-EU" device="C0805"/>
 <part name="SUPPLY2" library="supply2" deviceset="GND" device=""/>
+<part name="R6" library="resistor" deviceset="R-EU_" device="R0805"/>
+<part name="JP1" library="jumper" deviceset="JP1E" device=""/>
 </parts>
 <sheets>
@@
 <instance part="D3" gate="1" x="25.4" y="134.62" rot="R180"/>
 <instance part="D4" gate="1" x="25.4" y="81.28" rot="R180"/>
-<instance part="D5" gate="1" x="48.26" y="99.06" rot="R180"/>
+<instance part="D5" gate="1" x="48.26" y="93.98" rot="R90"/>
 <instance part="C14" gate="G$1" x="88.9" y="96.52"/>
 <instance part="C15" gate="G$1" x="83.82" y="124.46"/>
@@
 <instance part="C20" gate="G$1" x="86.36" y="152.4"/>
 <instance part="GND28" gate="1" x="83.82" y="142.24"/>
-<instance part="R5" gate="G$1" x="132.08" y="132.08" rot="R270"/>
+<instance part="0OHM" gate="G$1" x="132.08" y="132.08" rot="R270"/>
 <instance part="L8" gate="G$1" x="157.48" y="83.82"/>
 <instance part="L9" gate="G$1" x="157.48" y="68.58"/>
@@
 <instance part="C21" gate="G$1" x="152.4" y="76.2" rot="R90"/>
 <instance part="SUPPLY2" gate="GND" x="142.24" y="76.2" rot="R270"/>
+<instance part="R6" gate="G$1" x="58.42" y="142.24" rot="R90"/>
+<instance part="JP1" gate="A" x="137.16" y="142.24" rot="R270"/>
 </instances>
 <busses>
@@
 <pinref part="C11" gate="G$1" pin="2"/>
 <pinref part="GND13" gate="1" pin="GND"/>
+<pinref part="D5" gate="1" pin="A"/>
+<wire x1="53.34" y1="88.9" x2="48.26" y2="88.9" width="0.1524" layer="91"/>
+<wire x1="48.26" y1="88.9" x2="48.26" y2="91.44" width="0.1524" layer="91"/>
+<junction x="53.34" y="88.9"/>
 </segment>
 <segment>
@@
 <wire x1="40.64" y1="109.22" x2="40.64" y2="99.06" width="0.1524" layer="91"/>
 <wire x1="40.64" y1="99.06" x2="35.56" y2="99.06" width="0.1524" layer="91"/>
-<wire x1="45.72" y1="99.06" x2="40.64" y2="99.06" width="0.1524" layer="91"/>
 <pinref part="D2" gate="1" pin="A"/>
 <pinref part="C5" gate="G$1" pin="1"/>
 <pinref part="IC2" gate="A1" pin="VO"/>
 <pinref part="D5" gate="1" pin="C"/>
+<wire x1="40.64" y1="99.06" x2="48.26" y2="99.06" width="0.1524" layer="91"/>
+<wire x1="48.26" y1="99.06" x2="48.26" y2="96.52" width="0.1524" layer="91"/>
+<junction x="40.64" y="99.06"/>
+<wire x1="53.34" y1="99.06" x2="58.42" y2="99.06" width="0.1524" layer="91"/>
+<pinref part="L3" gate="G$1" pin="1"/>
+<pinref part="C11" gate="G$1" pin="1"/>
+<wire x1="48.26" y1="99.06" x2="53.34" y2="99.06" width="0.1524" layer="91"/>
+<junction x="48.26" y="99.06"/>
+<junction x="53.34" y="99.06"/>
 </segment>
 </net>
@@
 </segment>
 </net>
-<net name="N$14" class="0">
-<segment>
-<wire x1="53.34" y1="99.06" x2="58.42" y2="99.06" width="0.1524" layer="91"/>
-<wire x1="53.34" y1="99.06" x2="50.8" y2="99.06" width="0.1524" layer="91"/>
-<junction x="53.34" y="99.06"/>
-<pinref part="L3" gate="G$1" pin="1"/>
-<pinref part="C11" gate="G$1" pin="1"/>
-<pinref part="D5" gate="1" pin="A"/>
-</segment>
-</net>
 <net name="N$2" class="0">
 <segment>
@@
 <pinref part="IC4" gate="1" pin="AVCC"/>
 <pinref part="IC4" gate="1" pin="AREF"/>
-</segment>
-</net>
-<net name="N$9" class="0">
-<segment>
-<wire x1="137.16" y1="200.66" x2="137.16" y2="198.12" width="0.1524" layer="91"/>
-<wire x1="127" y1="200.66" x2="137.16" y2="200.66" width="0.1524" layer="91"/>
-<wire x1="127" y1="160.02" x2="127" y2="200.66" width="0.1524" layer="91"/>
-<wire x1="58.42" y1="162.56" x2="58.42" y2="160.02" width="0.1524" layer="91"/>
-<wire x1="58.42" y1="160.02" x2="58.42" y2="132.08" width="0.1524" layer="91"/>
-<wire x1="58.42" y1="160.02" x2="127" y2="160.02" width="0.1524" layer="91"/>
-<junction x="58.42" y="160.02"/>
-<pinref part="SV1" gate="G$1" pin="5"/>
-<pinref part="IC4" gate="1" pin="PC6(/RESET/PCINT14)"/>
-<pinref part="SV1" gate="G$1" pin="2"/>
-<wire x1="132.08" y1="182.88" x2="132.08" y2="137.16" width="0.1524" layer="91"/>
-<pinref part="L7" gate="G$1" pin="2"/>
-<pinref part="IC4" gate="1" pin="VCC@1"/>
-<wire x1="86.36" y1="154.94" x2="86.36" y2="162.56" width="0.1524" layer="91"/>
-<pinref part="C20" gate="G$1" pin="1"/>
-<junction x="86.36" y="154.94"/>
-<pinref part="IC4" gate="1" pin="VCC@2"/>
-<wire x1="88.9" y1="162.56" x2="88.9" y2="154.94" width="0.1524" layer="91"/>
-<wire x1="88.9" y1="154.94" x2="86.36" y2="154.94" width="0.1524" layer="91"/>
-<junction x="88.9" y="154.94"/>
-<wire x1="88.9" y1="154.94" x2="88.9" y2="132.08" width="0.1524" layer="91"/>
-<wire x1="93.98" y1="132.08" x2="88.9" y2="132.08" width="0.1524" layer="91"/>
-<junction x="93.98" y="132.08"/>
-<pinref part="C19" gate="G$1" pin="1"/>
-<wire x1="93.98" y1="132.08" x2="93.98" y2="137.16" width="0.1524" layer="91"/>
-<wire x1="93.98" y1="137.16" x2="93.98" y2="144.78" width="0.1524" layer="91"/>
-<junction x="93.98" y="137.16"/>
-<wire x1="93.98" y1="137.16" x2="132.08" y2="137.16" width="0.1524" layer="91"/>
-<junction x="132.08" y="137.16"/>
-<pinref part="R5" gate="G$1" pin="1"/>
-<wire x1="58.42" y1="132.08" x2="88.9" y2="132.08" width="0.1524" layer="91"/>
-<junction x="88.9" y="132.08"/>
 </segment>
 </net>
@@
 <net name="N$11" class="0">
 <segment>
-<pinref part="R5" gate="G$1" pin="2"/>
+<pinref part="0OHM" gate="G$1" pin="2"/>
 <pinref part="L6" gate="G$1" pin="2"/>
 <wire x1="88.9" y1="76.2" x2="91.44" y2="76.2" width="0.1524" layer="91"/>
@@
 </segment>
 </net>
+<net name="N$14" class="0">
+<segment>
+<pinref part="IC4" gate="1" pin="PC6(/RESET/PCINT14)"/>
+<pinref part="R6" gate="G$1" pin="2"/>
+<wire x1="58.42" y1="147.32" x2="58.42" y2="152.4" width="0.1524" layer="91"/>
+<pinref part="SV1" gate="G$1" pin="5"/>
+<wire x1="58.42" y1="152.4" x2="58.42" y2="162.56" width="0.1524" layer="91"/>
+<wire x1="137.16" y1="200.66" x2="137.16" y2="198.12" width="0.1524" layer="91"/>
+<wire x1="127" y1="200.66" x2="137.16" y2="200.66" width="0.1524" layer="91"/>
+<wire x1="127" y1="152.4" x2="127" y2="200.66" width="0.1524" layer="91"/>
+<wire x1="58.42" y1="152.4" x2="127" y2="152.4" width="0.1524" layer="91"/>
+<junction x="58.42" y="152.4"/>
+</segment>
+</net>
+<net name="N$9" class="0">
+<segment>
+<pinref part="0OHM" gate="G$1" pin="1"/>
+<wire x1="134.62" y1="139.7" x2="132.08" y2="139.7" width="0.1524" layer="91"/>
+<wire x1="132.08" y1="139.7" x2="132.08" y2="137.16" width="0.1524" layer="91"/>
+<pinref part="JP1" gate="A" pin="2"/>
+</segment>
+</net>
+<net name="N$27" class="0">
+<segment>
+<pinref part="SV1" gate="G$1" pin="2"/>
+<wire x1="132.08" y1="182.88" x2="132.08" y2="142.24" width="0.1524" layer="91"/>
+<pinref part="JP1" gate="A" pin="1"/>
+<wire x1="134.62" y1="142.24" x2="132.08" y2="142.24" width="0.1524" layer="91"/>
+<wire x1="58.42" y1="137.16" x2="58.42" y2="132.08" width="0.1524" layer="91"/>
+<pinref part="L7" gate="G$1" pin="2"/>
+<pinref part="IC4" gate="1" pin="VCC@1"/>
+<wire x1="86.36" y1="154.94" x2="86.36" y2="162.56" width="0.1524" layer="91"/>
+<pinref part="C20" gate="G$1" pin="1"/>
+<junction x="86.36" y="154.94"/>
+<pinref part="IC4" gate="1" pin="VCC@2"/>
+<wire x1="88.9" y1="162.56" x2="88.9" y2="154.94" width="0.1524" layer="91"/>
+<wire x1="88.9" y1="154.94" x2="86.36" y2="154.94" width="0.1524" layer="91"/>
+<junction x="88.9" y="154.94"/>
+<wire x1="88.9" y1="154.94" x2="88.9" y2="132.08" width="0.1524" layer="91"/>
+<wire x1="93.98" y1="132.08" x2="88.9" y2="132.08" width="0.1524" layer="91"/>
+<junction x="93.98" y="132.08"/>
+<pinref part="C19" gate="G$1" pin="1"/>
+<wire x1="93.98" y1="132.08" x2="93.98" y2="139.7" width="0.1524" layer="91"/>
+<wire x1="93.98" y1="142.24" x2="93.98" y2="144.78" width="0.1524" layer="91"/>
+<wire x1="58.42" y1="132.08" x2="88.9" y2="132.08" width="0.1524" layer="91"/>
+<junction x="88.9" y="132.08"/>
+<pinref part="R6" gate="G$1" pin="1"/>
+<wire x1="132.08" y1="142.24" x2="93.98" y2="142.24" width="0.1524" layer="91"/>
+<wire x1="93.98" y1="142.24" x2="93.98" y2="139.7" width="0.1524" layer="91"/>
+<junction x="132.08" y="142.24"/>
+</segment>
+</net>

Commit message: new version of braeburn for new board_port_connector
Parts:
- removed 0OHM: (no value), rcl:R-EU_0411/15
- removed C21: (no value), rcl:C-EUC0805
- removed JP1: (no value), jumper:JP1E
- removed L8, L9: (no value), rcl:L-EU0207/5V
- removed LED1: (no value), led:LED3MM
- removed R4: (no value), rcl:R-EU_R2012
- removed X2: (no value), con-wago-508:W237-04P
- removed X3: (no value), con-weidmueller-sl35:180G-6
- removed X4: (no value), con-wago-500:W237-102
- added IC6: MAX481CSA, maxim:MAX481CSA
- added U$2: HGG_LOGO, hgg:HGG_LOGO
- C14, C15, C16: device capacitor-wima:C5/7.2 -> capacitor-wima:C2.5/6
- U$1: value FRIENDSHIPEDGECONNECTOR -> FRIENDSHIPCONNECTOR; device hgg:FRIENDSHIPEDGECONNECTOR -> hgg:FRIENDSHIPCONNECTOR
Connections:
- removed net N$10: C14.1, L4.2, R2.2, X2-3.KL
- removed net N$11: 0OHM.2, C16.1, L6.2, L8.1, LED1.A, R3.2, X2-4.KL
- removed net N$19: LED1.C, R4.1
- removed net N$21: IC4.PD1(TXD/PCINT17), X3.2
- removed net N$22: IC4.PD0(RXD/PCINT16), X3.3
- removed net N$23: IC4.PC5(ADC5/SCL/PCINT13), X3.4
- removed net N$24: IC4.PC4(ADC4/SDA/PCINT12), X3.5
- removed net N$25: IC4.PC3(ADC3/PCINT11), X3.6
- removed net N$27: C19.1, C20.1, IC4.VCC@1, IC4.VCC@2, JP1.1, L7.2, R6.1, SV1.2
- removed net N$28: C15.1, L2.2, R1.2, X2-2.KL
- removed net N$29: C21.2, L8.2, L9.1
- removed net N$30: L9.2, X4-1.KL
- removed net N$9: 0OHM.1, JP1.2
- new net +12V: C15.1, L2.2, R1.2, U$1.+12V_A, U$1.+12V_B
- new net +3V3: C14.1, C19.1, C20.1, IC4.VCC@1, IC4.VCC@2, IC6P.GND, L4.2, L7.2, R2.2, R6.1, SV1.2, U$1.+3V3_A, U$1.+3V3_B
- new net +5V: C16.1, L6.2, R3.2, U$1.+5V_A, U$1.+5V_B
- new net BUS0+: IC6G$1.A, U$1.BUS0+
- new net BUS0-: IC6G$1.B, U$1.BUS0-
- new net BUSCTL: IC4.PC5(ADC5/SCL/PCINT13), IC6G$1.DE, IC6G$1.RE/
- new net CS: IC4.PD2(INT0/PCINT18), U$1./CS,IRQ
- new net IRQ: IC4.PC4(ADC4/SDA/PCINT12), U$1.IRQ
- new net N$34: U$1.PRSNT1, U$1.PRSNT2
- new net RX: IC4.PD0(RXD/PCINT16), IC6G$1.RO
- new net SLOWTIMECLK: IC4.PC1(ADC1/PCINT9), U$1.SLOWCLKCLK
- new net SLOWTIMECS: IC4.PC2(ADC2/PCINT10), U$1.SLOWCLK/CS
- new net SLOWTIMEMOSI: IC4.PC0(ADC0/PCINT8), U$1.SLOWCLKMOSI
- new net TX: IC4.PD1(TXD/PCINT17), IC6G$1.DI
- net GND: now also IC6P.VCC, U$1.GND1_A, U$1.GND1_B, U$1.GND2_A, U$1.GND2_B, U$1.GND3_A, U$1.GND3_B, U$1.GND4, U$1.GND5, U$1.GND7; no longer C21.1, R4.2, X2-1.KL, X4-2.KL
- net N$20: now also U$1.TDO, U$1.TMS; no longer IC4.PD2(INT0/PCINT18), X3.1
Other:
- note added: "+3V3"
- note added: "BUS0+"
- note added: "BUS0-"
- note added: "CS"
- note added: "IRQ"
- note added: "RS485CTL"
- note added: "RX"
- note added: "SLOWTIMECLK"
- note added: "SLOWTIMECS"
- note added: "SLOWTIMEMOSI"
- note added: "TX"
- note removed: "+3.3V"
- note removed: "GND"
- moved on the sheet: C17, C18, Q1

Commit message: current status
Parts:
- added IC5, IC7: LM741D, linear:LM741D
Connections:
- new net 3V3A: C11.1, C5.1, D2.A, D5.C, IC2.VO, IC5.+IN, L3.1
- new net 3V3B: C4.1, IC5.-IN, L3.2, L4.1
- new net 3V3METER: IC4.ADC6, IC5.OUT
- new net 5VA: C12.1, C8.1, D4.A, IC3.VO, IC7.+IN, L5.1
- new net 5VB: C9.1, IC7.-IN, L5.2, L6.1
- new net 5VMETER: IC4.ADC7, IC7.OUT
- net GND: now also IC5.ON1, IC5.ON2, IC5.V-, IC7.ON1, IC7.ON2, IC7.V-, U$1.GND6
- net N$3: now also IC7.V+; no longer C12.1, C8.1, D4.A, IC3.VO, L5.1
- net N$4: now also IC7.OPT; no longer C11.1, C5.1, D2.A, D5.C, IC2.VO, L3.1
- net N$6: now also IC5.V+; no longer C9.1, L5.2, L6.1
- net N$7: now also IC5.OPT; no longer C4.1, L3.2, L4.1
Other:
- note added: "3V3A"
- note added: "3V3B"
- note added: "3V3Meter"
- note added: "5VA"
- note added: "5VB"
- note added: "5VMeter"
- moved on the sheet: C17, C18, C19, C20, IC4, IC6, IC6P, L7, Q1, R6, SV1

Commit message: .
Connections:
- removed net N$3: IC7.V+
- removed net N$4: IC7.OPT
- removed net N$6: IC5.V+
- removed net N$7: IC5.OPT
Changed lines of the file:
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@@
 <wire x1="66.04" y1="180.34" x2="66.04" y2="190.5" width="0.1524" layer="91"/>
 <wire x1="144.78" y1="228.6" x2="144.78" y2="226.06" width="0.1524" layer="91"/>
-<wire x1="134.62" y1="228.6" x2="144.78" y2="228.6" width="0.1524" layer="91"/>
-<wire x1="134.62" y1="180.34" x2="134.62" y2="228.6" width="0.1524" layer="91"/>
-<wire x1="66.04" y1="180.34" x2="134.62" y2="180.34" width="0.1524" layer="91"/>
+<wire x1="71.12" y1="228.6" x2="144.78" y2="228.6" width="0.1524" layer="91"/>
+<wire x1="71.12" y1="180.34" x2="71.12" y2="228.6" width="0.1524" layer="91"/>
+<wire x1="66.04" y1="180.34" x2="71.12" y2="180.34" width="0.1524" layer="91"/>
 <junction x="66.04" y="180.34"/>
 </segment>
@@
 </segment>
 </net>
-<net name="N$3" class="0">
-<segment>
-<pinref part="IC7" gate="A" pin="V+"/>
-<wire x1="-20.32" y1="231.14" x2="-20.32" y2="236.22" width="0.1524" layer="91"/>
-</segment>
-</net>
-<net name="N$4" class="0">
-<segment>
-<pinref part="IC7" gate="A" pin="OPT"/>
-<wire x1="-17.78" y1="215.9" x2="-17.78" y2="213.36" width="0.1524" layer="91"/>
-</segment>
-</net>
-<net name="N$6" class="0">
-<segment>
-<pinref part="IC5" gate="A" pin="V+"/>
-<wire x1="-20.32" y1="200.66" x2="-20.32" y2="203.2" width="0.1524" layer="91"/>
-</segment>
-</net>
-<net name="N$7" class="0">
-<segment>
-<pinref part="IC5" gate="A" pin="OPT"/>
-<wire x1="-17.78" y1="185.42" x2="-17.78" y2="182.88" width="0.1524" layer="91"/>
-</segment>
-</net>

Commit message: slight update
Connections:
- net +3V3: now also IC5.V+, IC7.V+
Changed lines of the file:
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@@
 <text x="58.42" y="81.28" size="1.778" layer="91">5VA</text>
 <text x="73.66" y="81.28" size="1.778" layer="91">5VB</text>
+<text x="-20.32" y="233.68" size="1.778" layer="91" rot="R90">+3V3</text>
+<text x="-20.32" y="203.2" size="1.778" layer="91" rot="R90">+3V3</text>
 </plain>
 <instances>
@@
 <pinref part="IC6" gate="P" pin="GND"/>
 </segment>
+<segment>
+<pinref part="IC7" gate="A" pin="V+"/>
+<wire x1="-20.32" y1="231.14" x2="-20.32" y2="236.22" width="0.1524" layer="91"/>
+</segment>
+<segment>
+<pinref part="IC5" gate="A" pin="V+"/>
+<wire x1="-20.32" y1="200.66" x2="-20.32" y2="205.74" width="0.1524" layer="91"/>
+</segment>
 </net>
