File: hardware/braeburn/braeburn1/braeburn.sch (EAGLE design)
At the start: 32 parts, among them IC1 MAX481CSA, IC2 MEGA8-AI, IC3 MAX4105EUK, IC4 MAX4105EUK, IC5 MAX4105EUK, X1 5566-20

Commit message: braeburn version
Parts:
- added D1: 3V3, diode:1N4728
- added JP3: AVR-ISP-6VERT, avr-7:AVR-ISP-6VERT
- added JP4: (no value), pinhead:PINHD-1X2
- added R3: (no value), rcl:R-EU_R0603
- added SJ1, SJ2: (no value), jumper:SJW
- added U$2: HGG_LOGO, hgg:HGG_LOGO
- added X2: (no value), con-molex:KK-156-4
- C13: value (none) -> 100nF
- Q1: value (none) -> 16-20MHz
Connections:
- removed net N$16: IC3P.VEE, IC4P.VEE
- removed net N$7: IC2.PB5(SCK)
- removed net VCC: C10.1, IC1P.VCC, R1.2
- new net MISO: IC2.PB4(MISO), JP3.1
- new net MOSI: IC2.PB3(MOSI/OC2), JP3.4
- new net N$15: D1.A, SJ1.1, SJ2.1
- new net SCK: IC2.PB5(SCK), JP3.3
- net AVCC: no longer IC2.AREF
- net GND: now also D1.C, JP3.6, JP4.1, X2-2.S, X2-3.S
- net IN_+12V: now also X2-4.S
- net IN_+3V3: now also X1-1.S
- net IN_+5V: now also R3.2, SJ2.2, X2-1.S
- net IN_-5V: now also IC3P.VEE, IC4P.VEE
- net MEASURE_12V: now also IC2.PC0(ADC0); no longer IC2.PC2(ADC2)
- net MEASURE_3V3: now also IC2.PC2(ADC2); no longer IC2.PC0(ADC0)
- net N$8: now also JP4.2, R3.1; no longer IC2.PB4(MISO)
- net OUT_+3V3: now also C10.1, IC1P.VCC, JP3.2, R1.2, SJ1.2
- net OUT_+5V: now also IC2.AREF
- net R/W: now also IC2.PC3(ADC3)
- net RST: now also JP3.5
Other:
- note added: "Define +3V3"
- note added: "PWRLED"
- moved on the sheet: JP1, JP2, R1, X1-1, X1-10, X1-11, X1-12, X1-13, X1-14, X1-15, X1-16, X1-17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

Commit message: new braeburn version for using a PC ps
Parts:
- removed U$2: HGG_LOGO, hgg:HGG_LOGO
Changed lines of the file:
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@@
 <grid distance="0.1" unitdist="inch" unit="inch" style="lines" multiple="1" display="no" altdistance="0.01" altunitdist="inch" altunit="inch"/>
 <layers>
-<layer number="1" name="Top" color="4" fill="1" visible="yes" active="no"/>
-<layer number="16" name="Bottom" color="1" fill="1" visible="yes" active="no"/>
-<layer number="17" name="Pads" color="2" fill="1" visible="yes" active="no"/>
-<layer number="18" name="Vias" color="2" fill="1" visible="yes" active="no"/>
-<layer number="19" name="Unrouted" color="6" fill="1" visible="yes" active="no"/>
-<layer number="20" name="Dimension" color="15" fill="1" visible="yes" active="no"/>
-<layer number="21" name="tPlace" color="7" fill="1" visible="yes" active="no"/>
-<layer number="22" name="bPlace" color="7" fill="1" visible="yes" active="no"/>
-<layer number="23" name="tOrigins" color="15" fill="1" visible="yes" active="no"/>
-<layer number="24" name="bOrigins" color="15" fill="1" visible="yes" active="no"/>
-<layer number="25" name="tNames" color="7" fill="1" visible="yes" active="no"/>
-<layer number="26" name="bNames" color="7" fill="1" visible="yes" active="no"/>
-<layer number="27" name="tValues" color="7" fill="1" visible="yes" active="no"/>
-<layer number="28" name="bValues" color="7" fill="1" visible="yes" active="no"/>
+<layer number="1" name="Top" color="4" fill="1" visible="no" active="no"/>
+<layer number="16" name="Bottom" color="1" fill="1" visible="no" active="no"/>
+<layer number="17" name="Pads" color="2" fill="1" visible="no" active="no"/>
+<layer number="18" name="Vias" color="2" fill="1" visible="no" active="no"/>
+<layer number="19" name="Unrouted" color="6" fill="1" visible="no" active="no"/>
+<layer number="20" name="Dimension" color="15" fill="1" visible="no" active="no"/>
+<layer number="21" name="tPlace" color="7" fill="1" visible="no" active="no"/>
+<layer number="22" name="bPlace" color="7" fill="1" visible="no" active="no"/>
+<layer number="23" name="tOrigins" color="15" fill="1" visible="no" active="no"/>
+<layer number="24" name="bOrigins" color="15" fill="1" visible="no" active="no"/>
+<layer number="25" name="tNames" color="7" fill="1" visible="no" active="no"/>
+<layer number="26" name="bNames" color="7" fill="1" visible="no" active="no"/>
+<layer number="27" name="tValues" color="7" fill="1" visible="no" active="no"/>
+<layer number="28" name="bValues" color="7" fill="1" visible="no" active="no"/>
 <layer number="29" name="tStop" color="7" fill="3" visible="no" active="no"/>
 <layer number="30" name="bStop" color="7" fill="6" visible="no" active="no"/>
@@
 <layer number="35" name="tGlue" color="7" fill="4" visible="no" active="no"/>
 <layer number="36" name="bGlue" color="7" fill="5" visible="no" active="no"/>
-<layer number="37" name="tTest" color="7" fill="1" visible="yes" active="no"/>
-<layer number="38" name="bTest" color="7" fill="1" visible="yes" active="no"/>
+<layer number="37" name="tTest" color="7" fill="1" visible="no" active="no"/>
+<layer number="38" name="bTest" color="7" fill="1" visible="no" active="no"/>
 <layer number="39" name="tKeepout" color="4" fill="11" visible="no" active="no"/>
 <layer number="40" name="bKeepout" color="1" fill="11" visible="no" active="no"/>
@@
 <layer number="44" name="Drills" color="7" fill="1" visible="no" active="no"/>
 <layer number="45" name="Holes" color="7" fill="1" visible="no" active="no"/>
-<layer number="46" name="Milling" color="3" fill="1" visible="yes" active="no"/>
-<layer number="47" name="Measures" color="7" fill="1" visible="yes" active="no"/>
-<layer number="48" name="Document" color="7" fill="1" visible="yes" active="no"/>
-<layer number="49" name="Reference" color="7" fill="1" visible="yes" active="no"/>
-<layer number="50" name="dxf" color="7" fill="1" visible="yes" active="no"/>
-<layer number="51" name="tDocu" color="7" fill="1" visible="yes" active="no"/>
-<layer number="52" name="bDocu" color="7" fill="1" visible="yes" active="no"/>
+<layer number="46" name="Milling" color="3" fill="1" visible="no" active="no"/>
+<layer number="47" name="Measures" color="7" fill="1" visible="no" active="no"/>
+<layer number="48" name="Document" color="7" fill="1" visible="no" active="no"/>
+<layer number="49" name="Reference" color="7" fill="1" visible="no" active="no"/>
+<layer number="50" name="dxf" color="7" fill="1" visible="no" active="no"/>
+<layer number="51" name="tDocu" color="7" fill="1" visible="no" active="no"/>
+<layer number="52" name="bDocu" color="7" fill="1" visible="no" active="no"/>
 <layer number="91" name="Nets" color="2" fill="1" visible="yes" active="yes"/>
 <layer number="92" name="Busses" color="1" fill="1" visible="yes" active="yes"/>
@@
 <part name="GND17" library="supply1" deviceset="GND" device=""/>
 <part name="X2" library="con-molex" deviceset="KK-156-4" device=""/>
-<part name="U$2" library="hgg" deviceset="HGG_LOGO" device=""/>
 </parts>
 <sheets>
@@
 <instance part="X2" gate="-3" x="114.3" y="38.1"/>
 <instance part="X2" gate="-4" x="114.3" y="35.56"/>
-<instance part="U$2" gate="G$1" x="-83.82" y="63.5"/>
 </instances>
 <busses>
