File: hardware/braeburn/braeburn1/braeburn1.sch (EAGLE design)
At the start: 27 parts, among them IC1 MAX481CSA, IC2 MEGA8-AI, IC3 LM324D, Q1 20MHz

Commit message: new braeburn design
Parts:
- removed R3: (no value), rcl:R-EU_R0603
- added C10, C8, C9: (no value), rcl:C-EU025-050X050
- added C5, C6, C7: 22uF, rcl:C-EU025-050X050
- added D1, D2, D3: 11DQ06, diode:1N5817-B
- added IC4: LM2574N-12, linear:LM2574N-12
- added IC5: LM2574N-5.0, linear:LM2574N-5.0
- added IC6: LM2574N-3.3, linear:LM2574N-3.3
- added J2: (no value), con-jack:JACK-PLUG0
- added L1: (no value), rcl:L-EU0207/5V
- added L2, L3, L4: (no value), rcl:L-EUPIS2816
Connections:
- removed net N$15: R5.1
- removed net N$17: R14.1
- removed net N$19: R9.1
- new net DCIN: C5.1, C6.1, C7.1, IC4.IN, IC5.IN, IC6.IN, J2.3
- new net N$27: C9.2
- new net N_12V: D1.C, IC4.OUT, L3.1, R14.1
- new net N_3V3: D3.C, IC6.OUT, L4.1, R5.1
- new net N_5V: D2.C, IC5.OUT, L2.1, R9.1
- net AVCC: no longer R3.2
- net GND: now also C10.2, C5.2, C6.2, C7.2, C8.2, D1.A, D2.A, D3.A, IC4.!ON/OFF, IC4.GND@PWR, IC4.GNDSIG, IC5.!ON/OFF, IC5.GND@PWR, IC5.GNDSIG, IC6.!ON/OFF, IC6.GND@PWR, IC6.GNDSIG, J2.2
- net OUT_12V: now also C8.1, IC4.FB, L3.2
- net OUT_3V3: now also C10.1, IC6.FB, L1.1, L4.2; no longer R3.1
- net OUT_5V: now also C9.1, IC5.FB, L2.2
Other:
- note added: "SWITCHING REGULATORS"

Commit message: braeburn v1... so far
Parts:
- added C11, C12, C13: 10uF Kerko, rcl:C-EUC0603
- added C14, C15, C16: 2000uF, rcl:C-EU050-075X075
- C10, C8, C9: value (none) -> 220uF
Connections:
- removed net N$27: C9.2
- net AVCC: now also L1.2
- net GND: now also C11.2, C12.2, C13.2, C14.2, C15.2, C16.2, C9.2, R10.2
- net OUT_12V: now also C11.1, C14.1
- net OUT_3V3: now also C13.1, C16.1
- net OUT_5V: now also C12.1, C15.1
Other:
- moved on the sheet: C10, C8, C9, D1, D2, D3, IC4, IC5, L2, L3, L4

Commit message: improvements on the design
Parts:
- R16: value (none) -> 270Ohm
Connections:
- net OUT_3V3: no longer R16.1
- net OUT_5V: now also R16.1
Other:
- moved on the sheet: IC3A, IC3B, IC3C, R10, R11, R12, R13, R14, R15, R4, R5, R6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

Commit message: removed airwire.
Parts:
- added D4: 1N400X, diode:1N4004
Connections:
- new net N$15: D4.A, J2.3
- net DCIN: now also D4.C; no longer J2.3
- net GND: no longer U$1.GND2_B
Changed lines of the file:
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@@
 <part name="GND3" library="supply1" deviceset="GND" device=""/>
 <part name="GND4" library="supply1" deviceset="GND" device=""/>
-<part name="GND5" library="supply1" deviceset="GND" device=""/>
 <part name="GND6" library="supply1" deviceset="GND" device=""/>
 <part name="GND7" library="supply1" deviceset="GND" device=""/>
@@
 <part name="GND48" library="supply1" deviceset="GND" device=""/>
 <part name="GND49" library="supply1" deviceset="GND" device=""/>
+<part name="D4" library="diode" deviceset="1N4004" device="" value="1N400X"/>
 </parts>
 <sheets>
@@
 <instance part="GND3" gate="1" x="-5.08" y="55.88" rot="R270"/>
 <instance part="GND4" gate="1" x="104.14" y="55.88" rot="R90"/>
-<instance part="GND5" gate="1" x="104.14" y="60.96" rot="R90"/>
 <instance part="GND6" gate="1" x="104.14" y="66.04" rot="R90"/>
 <instance part="GND7" gate="1" x="-5.08" y="25.4" rot="R270"/>
@@
 <instance part="GND48" gate="1" x="218.44" y="-81.28"/>
 <instance part="GND49" gate="1" x="294.64" y="-81.28"/>
+<instance part="D4" gate="1" x="116.84" y="-111.76"/>
 </instances>
 <busses>
@@
 </segment>
 <segment>
-<pinref part="U$1" gate="G$1" pin="GND2_B"/>
-<wire x1="78.74" y1="60.96" x2="101.6" y2="60.96" width="0.1524" layer="91"/>
-<label x="88.9" y="60.96" size="1.778" layer="95"/>
-<pinref part="GND5" gate="1" pin="GND"/>
-</segment>
-<segment>
 <pinref part="U$1" gate="G$1" pin="GND3_B"/>
 <wire x1="78.74" y1="55.88" x2="101.6" y2="55.88" width="0.1524" layer="91"/>
@@
 </segment>
 <segment>
-<pinref part="J2" gate="G$1" pin="3"/>
-<wire x1="109.22" y1="-111.76" x2="134.62" y2="-111.76" width="0.1524" layer="91"/>
+<wire x1="119.38" y1="-111.76" x2="134.62" y2="-111.76" width="0.1524" layer="91"/>
 <label x="127" y="-111.76" size="1.778" layer="95"/>
+<pinref part="D4" gate="1" pin="C"/>
 </segment>
 </net>
@@
 </segment>
 </net>
+<net name="N$15" class="0">
+<segment>
+<pinref part="J2" gate="G$1" pin="3"/>
+<wire x1="109.22" y1="-111.76" x2="114.3" y2="-111.76" width="0.1524" layer="91"/>
+<pinref part="D4" gate="1" pin="A"/>
+</segment>
+</net>

Commit message: .
Parts:
- R16: value 270Ohm -> 330Ohm
Other:
- moved on the sheet: IC3A, R10, R12, R4, R5, R6, R7
Changed lines of the file:
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@@
 <part name="PWRLED" library="pinhead" deviceset="PINHD-1X2" device=""/>
 <part name="GND25" library="supply1" deviceset="GND" device=""/>
-<part name="R16" library="rcl" deviceset="R-EU_" device="R0603" value="270Ohm"/>
+<part name="R16" library="rcl" deviceset="R-EU_" device="R0603" value="330Ohm"/>
 <part name="L1" library="rcl" deviceset="L-EU" device="0207/5V"/>
 <part name="IC4" library="linear" deviceset="LM2574?-*" device="N" technology="12"/>
@@
 <instance part="GND18" gate="1" x="149.86" y="-12.7"/>
 <instance part="GND19" gate="1" x="149.86" y="15.24"/>
-<instance part="IC3" gate="A" x="35.56" y="-50.8"/>
+<instance part="IC3" gate="A" x="35.56" y="-48.26"/>
 <instance part="IC3" gate="B" x="35.56" y="-78.74"/>
 <instance part="IC3" gate="C" x="35.56" y="-109.22"/>
 <instance part="IC3" gate="P" x="30.48" y="-124.46" rot="R270"/>
 <instance part="GND20" gate="1" x="5.08" y="-124.46" rot="R270"/>
-<instance part="R4" gate="G$1" x="35.56" y="-58.42"/>
-<instance part="R5" gate="G$1" x="17.78" y="-53.34"/>
-<instance part="R6" gate="G$1" x="17.78" y="-48.26"/>
-<instance part="R7" gate="G$1" x="25.4" y="-43.18" rot="R90"/>
-<instance part="GND21" gate="1" x="15.24" y="-38.1" rot="R270"/>
+<instance part="R4" gate="G$1" x="35.56" y="-55.88"/>
+<instance part="R5" gate="G$1" x="17.78" y="-50.8"/>
+<instance part="R6" gate="G$1" x="17.78" y="-45.72"/>
+<instance part="R7" gate="G$1" x="25.4" y="-40.64" rot="R90"/>
+<instance part="GND21" gate="1" x="15.24" y="-35.56" rot="R270"/>
 <instance part="R8" gate="G$1" x="17.78" y="-76.2"/>
 <instance part="R9" gate="G$1" x="17.78" y="-81.28"/>
-<instance part="R10" gate="G$1" x="25.4" y="-68.58" rot="R90"/>
+<instance part="R10" gate="G$1" x="25.4" y="-71.12" rot="R90"/>
 <instance part="R11" gate="G$1" x="38.1" y="-86.36"/>
-<instance part="GND22" gate="1" x="15.24" y="-63.5" rot="R270"/>
-<instance part="R12" gate="G$1" x="25.4" y="-99.06" rot="R90"/>
+<instance part="GND22" gate="1" x="15.24" y="-66.04" rot="R270"/>
+<instance part="R12" gate="G$1" x="25.4" y="-101.6" rot="R90"/>
 <instance part="R13" gate="G$1" x="17.78" y="-106.68"/>
 <instance part="R14" gate="G$1" x="17.78" y="-111.76"/>
 <instance part="R15" gate="G$1" x="35.56" y="-116.84"/>
-<instance part="GND23" gate="1" x="15.24" y="-93.98" rot="R270"/>
+<instance part="GND23" gate="1" x="15.24" y="-96.52" rot="R270"/>
 <instance part="PWRLED" gate="G$1" x="99.06" y="35.56" rot="R90"/>
 <instance part="GND25" gate="1" x="96.52" y="12.7"/>
@@
 <segment>
 <pinref part="R6" gate="G$1" pin="1"/>
-<wire x1="12.7" y1="-48.26" x2="0" y2="-48.26" width="0.1524" layer="91"/>
-<label x="0" y="-48.26" size="1.778" layer="95"/>
+<wire x1="12.7" y1="-45.72" x2="0" y2="-45.72" width="0.1524" layer="91"/>
+<label x="0" y="-45.72" size="1.778" layer="95"/>
 </segment>
 <segment>
@@
 </segment>
 <segment>
-<wire x1="17.78" y1="-38.1" x2="25.4" y2="-38.1" width="0.1524" layer="91"/>
-<label x="33.02" y="-38.1" size="1.778" layer="95"/>
+<wire x1="17.78" y1="-35.56" x2="25.4" y2="-35.56" width="0.1524" layer="91"/>
+<label x="33.02" y="-35.56" size="1.778" layer="95"/>
 <pinref part="GND21" gate="1" pin="GND"/>
 <pinref part="R7" gate="G$1" pin="2"/>
-<junction x="25.4" y="-38.1"/>
-<wire x1="25.4" y1="-38.1" x2="38.1" y2="-38.1" width="0.1524" layer="91"/>
-</segment>
-<segment>
-<wire x1="17.78" y1="-63.5" x2="25.4" y2="-63.5" width="0.1524" layer="91"/>
+<junction x="25.4" y="-35.56"/>
+<wire x1="25.4" y1="-35.56" x2="38.1" y2="-35.56" width="0.1524" layer="91"/>
+</segment>
+<segment>
+<wire x1="17.78" y1="-66.04" x2="25.4" y2="-66.04" width="0.1524" layer="91"/>
 <pinref part="GND22" gate="1" pin="GND"/>
-<label x="33.02" y="-63.5" size="1.778" layer="95"/>
+<label x="33.02" y="-66.04" size="1.778" layer="95"/>
 <pinref part="R10" gate="G$1" pin="2"/>
-<wire x1="25.4" y1="-63.5" x2="38.1" y2="-63.5" width="0.1524" layer="91"/>
-</segment>
-<segment>
-<wire x1="17.78" y1="-93.98" x2="25.4" y2="-93.98" width="0.1524" layer="91"/>
-<label x="33.02" y="-93.98" size="1.778" layer="95"/>
+<wire x1="25.4" y1="-66.04" x2="38.1" y2="-66.04" width="0.1524" layer="91"/>
+</segment>
+<segment>
+<wire x1="17.78" y1="-96.52" x2="25.4" y2="-96.52" width="0.1524" layer="91"/>
+<label x="33.02" y="-96.52" size="1.778" layer="95"/>
 <pinref part="R12" gate="G$1" pin="2"/>
-<junction x="25.4" y="-93.98"/>
-<wire x1="25.4" y1="-93.98" x2="38.1" y2="-93.98" width="0.1524" layer="91"/>
+<junction x="25.4" y="-96.52"/>
+<wire x1="25.4" y1="-96.52" x2="38.1" y2="-96.52" width="0.1524" layer="91"/>
 <pinref part="GND23" gate="1" pin="GND"/>
 </segment>
@@
 <segment>
 <pinref part="IC3" gate="A" pin="OUT"/>
-<wire x1="43.18" y1="-50.8" x2="45.72" y2="-50.8" width="0.1524" layer="91"/>
-<wire x1="45.72" y1="-50.8" x2="63.5" y2="-50.8" width="0.1524" layer="91"/>
-<wire x1="40.64" y1="-58.42" x2="45.72" y2="-58.42" width="0.1524" layer="91"/>
-<wire x1="45.72" y1="-58.42" x2="45.72" y2="-50.8" width="0.1524" layer="91"/>
-<junction x="45.72" y="-50.8"/>
+<wire x1="43.18" y1="-48.26" x2="45.72" y2="-48.26" width="0.1524" layer="91"/>
+<wire x1="45.72" y1="-48.26" x2="63.5" y2="-48.26" width="0.1524" layer="91"/>
+<wire x1="40.64" y1="-55.88" x2="45.72" y2="-55.88" width="0.1524" layer="91"/>
+<wire x1="45.72" y1="-55.88" x2="45.72" y2="-48.26" width="0.1524" layer="91"/>
+<junction x="45.72" y="-48.26"/>
 <pinref part="R4" gate="G$1" pin="2"/>
-<label x="55.88" y="-50.8" size="1.778" layer="95"/>
+<label x="55.88" y="-48.26" size="1.778" layer="95"/>
 </segment>
 </net>
@@
 <pinref part="R5" gate="G$1" pin="2"/>
 <pinref part="IC3" gate="A" pin="-IN"/>
-<wire x1="22.86" y1="-53.34" x2="25.4" y2="-53.34" width="0.1524" layer="91"/>
+<wire x1="22.86" y1="-50.8" x2="25.4" y2="-50.8" width="0.1524" layer="91"/>
 <pinref part="R4" gate="G$1" pin="1"/>
-<wire x1="25.4" y1="-53.34" x2="27.94" y2="-53.34" width="0.1524" layer="91"/>
-<wire x1="30.48" y1="-58.42" x2="25.4" y2="-58.42" width="0.1524" layer="91"/>
-<wire x1="25.4" y1="-58.42" x2="25.4" y2="-53.34" width="0.1524" layer="91"/>
-<junction x="25.4" y="-53.34"/>
+<wire x1="25.4" y1="-50.8" x2="27.94" y2="-50.8" width="0.1524" layer="91"/>
+<wire x1="30.48" y1="-55.88" x2="25.4" y2="-55.88" width="0.1524" layer="91"/>
+<wire x1="25.4" y1="-55.88" x2="25.4" y2="-50.8" width="0.1524" layer="91"/>
+<junction x="25.4" y="-50.8"/>
 </segment>
 </net>
@@
 <pinref part="IC3" gate="A" pin="+IN"/>
 <pinref part="R6" gate="G$1" pin="2"/>
-<wire x1="27.94" y1="-48.26" x2="25.4" y2="-48.26" width="0.1524" layer="91"/>
+<wire x1="27.94" y1="-45.72" x2="25.4" y2="-45.72" width="0.1524" layer="91"/>
 <pinref part="R7" gate="G$1" pin="1"/>
-<wire x1="25.4" y1="-48.26" x2="22.86" y2="-48.26" width="0.1524" layer="91"/>
-<junction x="25.4" y="-48.26"/>
+<wire x1="25.4" y1="-45.72" x2="22.86" y2="-45.72" width="0.1524" layer="91"/>
+<junction x="25.4" y="-45.72"/>
 </segment>
 </net>
@@
 <pinref part="R10" gate="G$1" pin="1"/>
 <wire x1="25.4" y1="-76.2" x2="22.86" y2="-76.2" width="0.1524" layer="91"/>
-<wire x1="25.4" y1="-76.2" x2="25.4" y2="-73.66" width="0.1524" layer="91"/>
 <junction x="25.4" y="-76.2"/>
 </segment>
@@
 <pinref part="R12" gate="G$1" pin="1"/>
 <wire x1="25.4" y1="-106.68" x2="22.86" y2="-106.68" width="0.1524" layer="91"/>
-<wire x1="25.4" y1="-106.68" x2="25.4" y2="-104.14" width="0.1524" layer="91"/>
 <junction x="25.4" y="-106.68"/>
 </segment>
@@
 <segment>
 <pinref part="R5" gate="G$1" pin="1"/>
-<wire x1="12.7" y1="-53.34" x2="0" y2="-53.34" width="0.1524" layer="91"/>
-<label x="0" y="-53.34" size="1.778" layer="95"/>
-</segment>
-</net>
+<wire x1="12.7" y1="-50.8" x2="0" y2="-50.8" width="0.1524" layer="91"/>
+<label x="0" y="-50.8" size="1.778" layer="95"/>
+</segment>
+</net>
