File: hgg/modules/friendship/arduino_breakout/arduino_breakout.brd (EAGLE design)
At the start: 105.6 x 67.3 mm, 10 parts, among them IC1 MAX481CSA, IC2 MAX481CSA

Commit message: arduino breakout
Parts:
- added IC3, IC5, IC6: 74AC165D, 74xx-eu:SO16
- added IC4: 4517, 45xx:SO16
- added IC7, IC8, IC9: 74AC393D, 74xx-eu:SO14
Connections:
- net PA0 renamed N$38
- net PA1 renamed N$39
- net PA2 renamed N$18
- removed net PB6: JP6.6
- removed net PB7: JP6.5
- removed net VCC: C1.1, IC1.8, IC2.8
- new net FASTCLK3V3: IC7.1, U$1.A31(FASTCLK3V3)
- new net FASTTIMELATCH: IC3.1, IC5.1, IC6.1, JP6.5
- new net FASTTIMESHCLK: IC3.2, IC5.2, IC6.2, JP6.6
- new net N$10: IC3.11, IC7.3
- new net N$11: IC3.12, IC7.4
- new net N$12: IC3.14, IC7.13, IC7.6
- new net N$13: IC3.13, IC7.5
- new net N$14: IC3.3, IC7.11
- new net N$15: IC3.4, IC7.10
- new net N$16: IC3.5, IC7.9
- new net N$17: IC3.6, IC7.8, IC8.1
- new net N$19: IC6.6, IC9.8
- new net N$20: IC6.5, IC9.9
- new net N$21: IC6.4, IC9.10
- new net N$22: IC6.3, IC9.11
- new net N$23: IC6.14, IC9.6
- new net N$24: IC6.13, IC9.5
- new net N$25: IC6.12, IC9.4
- new net N$26: IC6.11, IC9.3
- new net N$27: IC5.6, IC8.8, IC9.1
- new net N$28: IC5.5, IC8.9
- new net N$29: IC5.4, IC8.10
- new net N$30: IC5.3, IC8.11
- new net N$31: IC5.14, IC8.13, IC8.6
- new net N$32: IC5.13, IC8.5
- new net N$33: IC4.5, IC4.9
- new net N$34: IC3.9, IC5.10
- new net N$35: IC5.12, IC8.4
- new net N$36: IC5.9, IC6.10
- new net N$37: IC5.11, IC8.3
- new net SLOWCLK/CS: IC4.13, IC4.3, U$1.A25(SLOWCLK/CS)
- new net SLOWCLKCLK: IC4.12, IC4.4, U$1.A24(SLOWCLKCLK)
- new net SLOWCLKMOSI: IC4.7, U$1.A23(SLOWTIMEMOSI)
- new net SLOWTIMESER: IC4.15
- net +5V: now also C1.1, IC1.8, IC2.8, IC3.16, IC4.16, IC5.16, IC6.16, IC7.14, IC8.14, IC9.14
- net GND: now also IC3.15, IC3.8, IC4.8, IC5.15, IC5.8, IC6.15, IC6.8, IC7.7, IC8.7, IC9.7
- net PPS: now also IC7.12, IC7.2, IC8.12, IC8.2, IC9.12, IC9.2
Routing:
- net +5V: track 143.0 -> 303.1 mm, vias 1 -> 6
- net FASTCLK3V3: track 0.00 -> 97.1 mm, vias 0 -> 3
- net SLOWCLK/CS: track 0.00 -> 64.4 mm, vias 0 -> 3
- net SLOWCLKCLK: track 0.00 -> 62.1 mm, vias 0 -> 3
- net SLOWCLKMOSI: track 0.00 -> 59.0 mm, vias 0 -> 3
- net SLOWTIMESER: track 0.00 -> 47.3 mm, vias 0 -> 3
- net PPS: track 77.5 -> 98.1 mm
- net N$24: track 0.00 -> 14.1 mm, vias 0 -> 1
- net N$26: track 0.00 -> 13.8 mm, vias 0 -> 1
- net N$37: track 0.00 -> 13.1 mm, vias 0 -> 1
- net N$19: track 0.00 -> 13.1 mm, vias 0 -> 1
- net N$20: track 0.00 -> 13.0 mm, vias 0 -> 1
- net N$21: track 0.00 -> 12.9 mm, vias 0 -> 1
- net N$22: track 0.00 -> 12.9 mm, vias 0 -> 1
- net VCC: track 12.8 -> 0.00 mm, vias 2 -> 0
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
Commit message: breakout
Parts:
- added C2, C3, C4, C5, C6, C7: 100nF, rcl:C0603
Connections:
- net PB5 renamed N$100
- removed net PH5: JP6.10
- net +5V: now also C2.1, C3.1, C4.1, C5.1, C6.1, C7.1
- net FASTCLK3V3: now also IC7.13; no longer IC7.1
- net GND: now also C2.2, C3.2, C4.2, C5.2, C6.2, C7.2
- net N$10: now also IC7.1, IC7.8; no longer IC3.11, IC7.3
- net N$11: now also IC3.13, IC7.9; no longer IC3.12, IC7.4
- net N$12: now also IC3.12, IC7.10; no longer IC3.14, IC7.13, IC7.6
- net N$13: now also IC3.11, IC7.11; no longer IC3.13, IC7.5
- net N$14: now also IC7.3; no longer IC7.11
- net N$15: now also IC7.4; no longer IC7.10
- net N$16: now also IC7.5; no longer IC7.9
- net N$17: now also IC7.6; no longer IC7.8
- net SLOWTIMESER: now also JP6.10
Routing:
- net PPS: track 98.1 -> 176.0 mm, vias 3 -> 8
- net FASTTIMELATCH: track 0.00 -> 76.8 mm, vias 0 -> 4
- net FASTTIMESHCLK: track 0.00 -> 72.2 mm, vias 0 -> 5
- net GND: track 272.0 -> 343.4 mm, vias 18 -> 36
- net N$17: track 0.00 -> 54.8 mm, vias 0 -> 4
- net N$27: track 12.1 -> 49.3 mm, vias 1 -> 3
- net SLOWTIMESER: track 47.3 -> 83.1 mm, vias 3 -> 4
- net +5V: track 303.1 -> 336.7 mm, vias 6 -> 9
- net FASTCLK3V3: track 97.1 -> 130.2 mm, vias 3 -> 5
- net N$36: track 0.00 -> 29.9 mm
- net N$31: track 11.5 -> 31.8 mm, vias 2 -> 3
- net N$14: track 0.00 -> 13.4 mm, vias 0 -> 1
- net N$16: track 0.00 -> 12.5 mm, vias 0 -> 1
- net N$23: track 9.85 -> 21.5 mm, vias 0 -> 1
- net N$15: track 0.00 -> 11.4 mm, vias 0 -> 1
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- added copper zone on layer 1, net GND
- added copper zone on layer 16, net GND
