File: hgg/modules/friendship/arduino_breakout/arduino_breakout.brd (EAGLE design)
At the start: 105.6 x 67.3 mm, 17 parts, among them IC1 MAX481CSA, IC2 MAX481CSA, IC3 74AC165D, IC4 4517, IC5 74AC165D, IC6 74AC165D, IC7 74AC393D, IC8 74AC393D, IC9 74AC393D

Commit message: breakout
Parts:
- added C2, C3, C4, C5, C6, C7: 100nF, rcl:C0603
Connections:
- removed net PB4: JP6.8
- removed net PB5: JP6.7
- removed net PH5: JP6.10
- net +5V: now also C2.1, C3.1, C4.1, C5.1, C6.1, C7.1
- net FASTCLK3V3: now also IC7.13; no longer IC7.1
- net GND: now also C2.2, C3.2, C4.2, C5.2, C6.2, C7.2
- net N$10: now also IC7.1, IC7.8; no longer IC3.11, IC7.3
- net N$11: now also IC3.13, IC7.9; no longer IC3.12, IC7.4
- net N$12: now also IC3.12, IC7.10; no longer IC3.14, IC7.13, IC7.6
- net N$13: now also IC3.11, IC7.11; no longer IC3.13, IC7.5
- net N$14: now also IC7.3; no longer IC7.11
- net N$15: now also IC7.4; no longer IC7.10
- net N$16: now also IC7.5; no longer IC7.9
- net N$17: now also IC7.6; no longer IC7.8
- net SLOWCLK/CS: now also JP6.8
- net SLOWCLKCLK: now also JP6.7
- net SLOWTIMESER: now also JP6.10
Routing:
- net PPS: track 98.1 -> 176.3 mm, vias 3 -> 8
- net FASTTIMELATCH: track 0.00 -> 77.1 mm, vias 0 -> 4
- net FASTTIMESHCLK: track 0.00 -> 72.2 mm, vias 0 -> 5
- net GND: track 272.0 -> 342.5 mm, vias 18 -> 36
- net N$17: track 0.00 -> 54.8 mm, vias 0 -> 4
- net SLOWCLKCLK: track 62.1 -> 103.1 mm, vias 3 -> 6
- net SLOWCLK/CS: track 64.4 -> 102.2 mm, vias 3 -> 6
- net N$27: track 12.1 -> 49.3 mm, vias 1 -> 3
- net SLOWTIMESER: track 47.3 -> 83.1 mm, vias 3 -> 4
- net +5V: track 303.1 -> 337.3 mm, vias 6 -> 9
- net FASTCLK3V3: track 97.1 -> 130.2 mm, vias 3 -> 5
- net N$36: track 0.00 -> 29.9 mm
- net N$31: track 11.5 -> 31.8 mm, vias 2 -> 3
- net N$14: track 0.00 -> 13.4 mm, vias 0 -> 1
- net N$16: track 0.00 -> 12.5 mm, vias 0 -> 1
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- added copper zone on layer 1, net GND
- added copper zone on layer 16, net GND
