File: hgg/modules/friendship/arduino_breakout/arduino_breakout.sch (EAGLE design)
At the start: 10 parts, among them IC1 MAX481CSA, IC2 MAX481CSA

Commit message: arduino breakout
Parts:
- added IC3, IC5, IC6: 74AC165D, 74xx-eu:74AC165D
- added IC4: 4517, 45xx:4517
- added IC7, IC8, IC9: 74AC393D, 74xx-eu:74AC393D
Connections:
- net PA0 renamed N$38
- net PA1 renamed N$39
- net PA2 renamed N$18
- removed net PB6: JP6.6
- removed net PB7: JP6.5
- removed net VCC: C1.1, IC1P.VCC, IC2P.VCC
- new net FASTCLK3V3: IC7A.A, U$1.FASTCLK3V3
- new net FASTTIMELATCH: IC3A.SH/!LD, IC5A.SH/!LD, IC6A.SH/!LD, JP6.5
- new net FASTTIMESHCLK: IC3A.CLK, IC5A.CLK, IC6A.CLK, JP6.6
- new net N$10: IC3A.A, IC7A.QA
- new net N$11: IC3A.B, IC7A.QB
- new net N$12: IC3A.D, IC7A.QD, IC7B.A
- new net N$13: IC3A.C, IC7A.QC
- new net N$14: IC3A.E, IC7B.QA
- new net N$15: IC3A.F, IC7B.QB
- new net N$16: IC3A.G, IC7B.QC
- new net N$17: IC3A.H, IC7B.QD, IC8A.A
- new net N$19: IC6A.H, IC9B.QD
- new net N$20: IC6A.G, IC9B.QC
- new net N$21: IC6A.F, IC9B.QB
- new net N$22: IC6A.E, IC9B.QA
- new net N$23: IC6A.D, IC9A.QD
- new net N$24: IC6A.C, IC9A.QC
- new net N$25: IC6A.B, IC9A.QB
- new net N$26: IC6A.A, IC9A.QA
- new net N$27: IC5A.H, IC8B.QD, IC9A.A
- new net N$28: IC5A.G, IC8B.QC
- new net N$29: IC5A.F, IC8B.QB
- new net N$30: IC5A.E, IC8B.QA
- new net N$31: IC5A.D, IC8A.QD, IC8B.A
- new net N$32: IC5A.C, IC8A.QC
- new net N$33: IC4A.Q64, IC4B.D
- new net N$34: IC3A.QH, IC5A.SER
- new net N$35: IC5A.B, IC8A.QB
- new net N$36: IC5A.QH, IC6A.SER
- new net N$37: IC5A.A, IC8A.QA
- new net SLOWCLK/CS: IC4A.WE, IC4B.WE, U$1.SLOWCLK/CS
- new net SLOWCLKCLK: IC4A.CLK, IC4B.CLK, U$1.SLOWCLKCLK
- new net SLOWCLKMOSI: IC4A.D, U$1.SLOWCLKMOSI
- new net SLOWTIMESER: IC4B.Q16
- net +5V: now also C1.1, IC1P.VCC, IC2P.VCC, IC3P.VCC, IC4P.VDD, IC5P.VCC, IC6P.VCC, IC7P.VCC, IC8P.VCC, IC9P.VCC
- net GND: now also IC3A.INH, IC3P.GND, IC4P.VSS, IC5A.INH, IC5P.GND, IC6A.INH, IC6P.GND, IC7P.GND, IC8P.GND, IC9P.GND
- net PPS: now also IC7A.CLR, IC7B.CLR, IC8A.CLR, IC8B.CLR, IC9A.CLR, IC9B.CLR
Other:
- moved on the sheet: IC1, IC2

Commit message: breakout
Parts:
- added C2, C3, C4, C5, C6, C7: 100nF, rcl:C-EUC0603
Connections:
- net PB5 renamed N$100
- removed net PH5: JP6.10
- net +5V: now also C2.1, C3.1, C4.1, C5.1, C6.1, C7.1
- net FASTCLK3V3: now also IC7B.A; no longer IC7A.A
- net GND: now also C2.2, C3.2, C4.2, C5.2, C6.2, C7.2
- net N$10: now also IC7A.A, IC7B.QD; no longer IC3A.A, IC7A.QA
- net N$11: now also IC3A.C, IC7B.QC; no longer IC3A.B, IC7A.QB
- net N$12: now also IC3A.B, IC7B.QB; no longer IC3A.D, IC7A.QD, IC7B.A
- net N$13: now also IC3A.A, IC7B.QA; no longer IC3A.C, IC7A.QC
- net N$14: now also IC7A.QA; no longer IC7B.QA
- net N$15: now also IC7A.QB; no longer IC7B.QB
- net N$16: now also IC7A.QC; no longer IC7B.QC
- net N$17: now also IC7A.QD; no longer IC7B.QD
- net SLOWTIMESER: now also JP6.10
Other:
- note added: "TODO: an chip anbinden"
- moved on the sheet: IC7A, IC7B
