File: hgg/modules/friendship/arduino_breakout/arduino_breakout.sch (EAGLE design)
At the start: 17 parts, among them IC1 MAX481CSA, IC2 MAX481CSA, IC3 74AC165D, IC4 4517, IC5 74AC165D, IC6 74AC165D, IC7 74AC393D, IC8 74AC393D, IC9 74AC393D

Commit message: breakout
Parts:
- added C2, C3, C4, C5, C6, C7: 100nF, rcl:C-EUC0603
Connections:
- removed net PB4: JP6.8
- removed net PB5: JP6.7
- removed net PH5: JP6.10
- net +5V: now also C2.1, C3.1, C4.1, C5.1, C6.1, C7.1
- net FASTCLK3V3: now also IC7B.A; no longer IC7A.A
- net GND: now also C2.2, C3.2, C4.2, C5.2, C6.2, C7.2
- net N$10: now also IC7A.A, IC7B.QD; no longer IC3A.A, IC7A.QA
- net N$11: now also IC3A.C, IC7B.QC; no longer IC3A.B, IC7A.QB
- net N$12: now also IC3A.B, IC7B.QB; no longer IC3A.D, IC7A.QD, IC7B.A
- net N$13: now also IC3A.A, IC7B.QA; no longer IC3A.C, IC7A.QC
- net N$14: now also IC7A.QA; no longer IC7B.QA
- net N$15: now also IC7A.QB; no longer IC7B.QB
- net N$16: now also IC7A.QC; no longer IC7B.QC
- net N$17: now also IC7A.QD; no longer IC7B.QD
- net SLOWCLK/CS: now also JP6.8
- net SLOWCLKCLK: now also JP6.7
- net SLOWTIMESER: now also JP6.10
Other:
- moved on the sheet: IC1, IC2, IC7A, IC7B

Commit message: small routing improvements
Connections:
- removed net PH6: JP6.9
- new net PH5: JP6.10
- net SLOWTIMESER: now also JP6.9; no longer JP6.10
Changed lines of the file:
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@@
 </segment>
 </net>
-<net name="PH6" class="0">
-<segment>
-<wire x1="99.06" y1="81.28" x2="119.38" y2="81.28" width="0.1524" layer="91"/>
-<label x="101.6" y="81.28" size="1.778" layer="95"/>
-<pinref part="JP6" gate="A" pin="9"/>
+<net name="PH5" class="0">
+<segment>
+<wire x1="99.06" y1="78.74" x2="119.38" y2="78.74" width="0.1524" layer="91"/>
+<label x="101.6" y="78.74" size="1.778" layer="95"/>
+<pinref part="JP6" gate="A" pin="10"/>
 </segment>
 </net>
@@
 </segment>
 <segment>
-<wire x1="119.38" y1="78.74" x2="99.06" y2="78.74" width="0.1524" layer="91"/>
-<label x="101.6" y="78.74" size="1.778" layer="95"/>
-<pinref part="JP6" gate="A" pin="10"/>
+<label x="101.6" y="81.28" size="1.778" layer="95"/>
+<pinref part="JP6" gate="A" pin="9"/>
+<wire x1="99.06" y1="81.28" x2="119.38" y2="81.28" width="0.1524" layer="91"/>
 </segment>
 </net>
@@
 <label x="101.6" y="91.44" size="1.6764" layer="95"/>
 <pinref part="JP6" gate="A" pin="5"/>
-<junction x="119.38" y="91.44"/>
 </segment>
 </net>
@@
 <label x="101.6" y="88.9" size="1.6764" layer="95"/>
 <pinref part="JP6" gate="A" pin="6"/>
-<junction x="119.38" y="88.9"/>
-</segment>
-</net>
+</segment>
+</net>
