File: hgg/modules/dash/testboards/miniadsb.brd (EAGLE design)
At the start: 39.7 x 46.3 mm, 16 parts, among them IC1 TLC272P, IC2 LM339N, IC3 7414N

Commit message: updates
Parts:
- added R7: 1k, rcl:R0603
Connections:
- net /ADSB_TTL: now also R7.1
- net VCC: now also R7.2
Routing:
- net /ADSB_TTL: track 10.5 -> 15.0 mm
- net VCC: track 101.6 -> 102.3 mm
Other:
- board size 39.7 x 46.3 mm -> 39.7 x 47.6 mm
Changed lines of the file:
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@@
 <plain>
 <wire x1="2.2225" y1="0" x2="41.8975" y2="0" width="0" layer="20"/>
-<wire x1="41.8975" y1="0" x2="41.8975" y2="46.345" width="0" layer="20"/>
-<wire x1="41.8975" y1="46.345" x2="2.2225" y2="46.345" width="0" layer="20"/>
-<wire x1="2.2225" y1="46.345" x2="2.2225" y2="0" width="0" layer="20"/>
+<wire x1="41.8975" y1="0" x2="41.8975" y2="47.615" width="0" layer="20"/>
+<wire x1="41.8975" y1="47.615" x2="2.2225" y2="47.615" width="0" layer="20"/>
+<wire x1="2.2225" y1="47.615" x2="2.2225" y2="0" width="0" layer="20"/>
 <text x="6.985" y="6.985" size="0.8128" layer="1" font="vector">hgg dash0 </text>
 <text x="6.985" y="5.715" size="0.8128" layer="1" font="vector">test board</text>
@@
 <element name="R6" library="resistor" package="R0805" value="330k" x="8.89" y="23.495"/>
 <element name="JP1" library="pinhead" package="1X04" value="" x="29.21" y="7.62" rot="R180"/>
+<element name="R7" library="rcl" package="R0603" value="1k" x="21.59" y="41.91" rot="R90"/>
 </elements>
 <signals>
@@
 <wire x1="18.9475" y1="20.0025" x2="22.23434375" y2="20.0025" width="0.8128" layer="1"/>
 <wire x1="22.23434375" y1="20.0025" x2="22.55184375" y2="20.32" width="0.8128" layer="1"/>
-<wire x1="17.4625" y1="43.18" x2="24.765" y2="43.18" width="0.8128" layer="1"/>
+<wire x1="17.4625" y1="43.18" x2="21.9075" y2="43.18" width="0.8128" layer="1"/>
+<wire x1="21.9075" y1="43.18" x2="24.765" y2="43.18" width="0.8128" layer="1"/>
 <wire x1="24.765" y1="43.18" x2="26.035" y2="41.91" width="0.8128" layer="1"/>
 <wire x1="26.035" y1="41.91" x2="28.8925" y2="41.91" width="0.8128" layer="1"/>
@@
 <wire x1="14.82" y1="42.545" x2="14.82" y2="42.33" width="0.8128" layer="1"/>
 <wire x1="14.82" y1="42.33" x2="14.9225" y2="42.2275" width="0.8128" layer="1"/>
+<contactref element="R7" pad="2"/>
+<wire x1="21.59" y1="42.76" x2="21.9075" y2="42.76" width="0.4064" layer="1"/>
+<wire x1="21.9075" y1="42.76" x2="21.9075" y2="43.18" width="0.4064" layer="1"/>
 </signal>
 <signal name="N$1">
@@
 <contactref element="IC3" pad="13"/>
 <wire x1="27.94" y1="40.64" x2="17.4625" y2="40.64" width="0.8128" layer="1"/>
+<contactref element="R7" pad="1"/>
+<wire x1="17.4625" y1="40.64" x2="21.59" y2="40.64" width="0.4064" layer="1"/>
+<wire x1="21.59" y1="40.64" x2="21.59" y2="41.06" width="0.4064" layer="1"/>
 </signal>
 <signal name="ADSB">
