File: hgg/modules/braeburn/braeburn1/braeburn1.sch (EAGLE design)
At the start: 50 parts, among them IC1 MAX481CSA, IC2 MEGA8-AI, IC3 LM324D, IC4 LM2574N-12, IC5 LM2574N-5.0, IC6 LM2574N-3.3, Q1 20MHz

Commit message: new release of braeburn board file
Parts:
- removed IC1: MAX481CSA, maxim:MAX481CSA
- added IC7: LTC485N, linear-technology:LTC485N
- added R17: 1k, rcl:R-EU_0207/12
- added R3: PTC-SOD70, ptc-ntc:PTC-SOD70
- Q1: value 20MHz -> 8-20MHz; device crystal:CRYSTALHC33U-V -> crystal:CRYSTALHC49S; OC_FARNELL (none) -> 1667008
- R1: value (none) -> 10k
Connections:
- removed net M_12V: IC3C.OUT, R15.2
- new net PTC: IC2.ADC7, R17.2, R3.2
- net BUS0+: now also IC7.B; no longer IC1G$1.A
- net BUS0-: now also IC7.A; no longer IC1G$1.B
- net GND: now also IC7.GND, R17.1; no longer IC1P.GND, U$1.GND1_B, U$1.GND3_B
- net M12V: now also IC3C.OUT, R15.2
- net N$4: now also Q1.1; no longer Q1.2
- net N$5: now also Q1.2; no longer Q1.1
- net OUT_12V: no longer U$1.+12V_A
- net OUT_3V3: now also IC7.VCC, R3.1; no longer IC1P.VCC, IC2.VCC@1, IC2.VCC@2, IC3P.V+, JP1.2, U$1.+3V3_A
- net OUT_5V: now also IC2.VCC@1, IC2.VCC@2, IC3P.V+, JP1.2; no longer U$1.+5V_A
- net RW: now also IC7.!RE, IC7.DE; no longer IC1G$1.DE, IC1G$1.RE/
- net RX: now also IC7.RO; no longer IC1G$1.RO
- net TX: now also IC7.DI; no longer IC1G$1.DI
Other:
- moved on the sheet: Q1
