File: hgg/modules/braeburn/braeburn0/power.sch (EAGLE design)
At the start: 54 parts, among them IC1 7812TV, IC2 7805TV, IC3 7805TV, IC4 ATMEGA48/88/168-AU

Commit message: new release of braeburn board file
Parts:
- removed 0OHM: (no value), rcl:R-EU_0411/15
- removed C21: (no value), rcl:C-EUC0805
- removed L8, L9: (no value), rcl:L-EU0207/5V
- removed X2: (no value), con-wago-508:W237-04P
- removed X3: (no value), con-weidmueller-sl35:180G-6
- removed X4: (no value), con-wago-500:W237-102
- added IC5: LTC485S, linear-technology:LTC485S
- added R5: 30K, rcl:R-EU_R0603
- C17, C18, C19, C20: device rcl:C-EUC0805 -> rcl:C-EUC0603
- R4: device rcl:R-EU_R2012 -> rcl:R-EU_R0603
- R6: device resistor:R-EU_R0805 -> resistor:R-EU_R0603
- U$1: value FRIENDSHIPEDGECONNECTOR -> FRIENDSHIPCONNECTOR; device hgg:FRIENDSHIPEDGECONNECTOR -> hgg:FRIENDSHIPCONNECTOR
Connections:
- new net N$31: C16.1, JP1.1, L6.2, R3.2, U$1.+5V_A, U$1.+5V_B
- new net N$32: IC4.PC2(ADC2/PCINT10), IC5.!RE, IC5.DE, R5.2
- new net N$33: IC4.PD3(INT1/OC2B/PCINT19), U$1./CS,IRQ
- new net N$34: IC4.PD4(T0/XCK/PCINT20), U$1.IRQ
- net GND: now also IC5.GND, U$1.GND1_A, U$1.GND1_B, U$1.GND2_A, U$1.GND2_B, U$1.GND3_A, U$1.GND3_B, U$1.GND4; no longer C21.1, X2-1.KL, X4-2.KL
- net N$10: now also IC5.VCC, R5.1, U$1.+3V3_A, U$1.+3V3_B; no longer X2-3.KL
- net N$11: now also IC5.A, U$1.BUS0-; no longer 0OHM.2, C16.1, L6.2, L8.1, LED1.A, R3.2, X2-4.KL
- net N$20: now also U$1.PPS; no longer X3.1
- net N$21: now also IC5.DI; no longer X3.2
- net N$22: now also IC5.B, U$1.BUS0+; no longer IC4.PD0(RXD/PCINT16), X3.3
- net N$23: now also U$1.PRSNT1, U$1.PRSNT2; no longer IC4.PC5(ADC5/SCL/PCINT13), X3.4
- net N$24: now also U$1.SLOWCLKCLK; no longer X3.5
- net N$25: now also U$1.SLOWCLKMOSI; no longer X3.6
- net N$27: no longer JP1.1
- net N$28: now also U$1.+12V_A, U$1.+12V_B; no longer X2-2.KL
- net N$29: now also U$1.TDI, U$1.TDO; no longer C21.2, L8.2, L9.1
- net N$30: now also IC4.PD0(RXD/PCINT16), IC5.RO; no longer L9.2, X4-1.KL
- net N$9: now also LED1.A; no longer 0OHM.1
Other:
- note removed: "GND"
- moved on the sheet: JP1, LED1, R4

Commit message: initial version of design update
Parts:
- removed C16: (no value), capacitor-wima:C5/7.2
- removed D5: 1N4728, diode:1N4728
- removed IC2, IC3: 7805TV, linear:7805TV
- removed L2, L4, L6: (no value), resistor:L-EU0207/5V
- added LED2, LED4: GM5BW96385A, led:GM5BW96385A
- added R10, R11, R12, R13, R14, R15, R16, R17, R18, R7, R8, R9: (no value), rcl:R-EU_R0603
- added R19, R20, R21: (no value), rcl:R-EU_0207/15
- added R22: PTC-SOD70, ptc-ntc:PTC-SOD70
- added R23, R24, R25: 2k, rcl:R-EU_R0603
- added U$2, U$3, U$4: AP1084, hgg:AP1084
- C13: value (none) -> 2000u
- C14: value (none) -> 100n; device capacitor-wima:C5/7.2 -> rcl:C-EUC0603
- C15: device capacitor-wima:C5/7.2 -> rcl:C-EUC0603
- C17, C18: value (none) -> 22n
- C19: value (none) -> 2n2
- C20: value (none) -> 100n
- IC1: value 7812TV -> LM324D; device linear:7812TV -> linear:LM324D
- L7: value (none) -> 33u
- R5: value 30K -> 10k
- R6: value (none) -> 10k
Connections:
- net N$11 renamed BUS0-
- net N$14 renamed RST
- net N$22 renamed BUS0+
- net N$33 renamed /CS
- net N$34 renamed IRQ
- removed net N$31: C16.1, JP1.1, L6.2, R3.2, U$1.+5V_A, U$1.+5V_B
- new net 12V: R16.1, R21.2, U$1.+12V_A, U$1.+12V_B
- new net 12VIN: C9.1, L5.2, R17.1, R21.1, R3.2
- new net 3V3: R19.2, R7.1, U$1.+3V3_A, U$1.+3V3_B
- new net 3V3IN: C3.1, L1.2, R1.2, R19.1, R9.1
- new net LED1: IC4.PD5(T1/OC0B/PCINT21), LED2.A
- new net LED2: IC4.PD6(AIN0/OC0A/PCINT22), LED4.A
- new net N$11: IC1B.OUT, R13.2
- new net N$14: IC1B.-IN, R12.2, R14.2
- new net N$22: IC1B.+IN, R11.2, R13.1
- new net N$26: IC1C.+IN, R15.1, R16.2
- new net N$36: LED2.C, R24.1
- new net N$37: LED4.C, R25.1
- new net TEMP1: IC4.ADC6, R22.2, R23.2
- new net VCC: C14.2, C15.2, C19.1, C20.1, IC1P.V+, IC4.VCC@1, IC4.VCC@2, IC5.VCC, JP1.1, L7.2, R11.1, R20.2, R23.1, R5.1, R6.1, SV1.2, U$1.+5V_A, U$1.+5V_B
- new net VCCIN: C4.1, L3.2, R12.1, R2.2, R20.1
- net GND: now also C14.1, C15.1, IC1P.V-, R10.1, R14.1, R18.1, R22.1, R24.2, R25.2, U$2.GND, U$3.GND, U$4.GND; no longer C14.2, C15.2, C16.2, D5.A, IC1.GND, IC2.GND, IC3.GND
- net N$1: now also U$2.VIN, U$3.VIN, U$4.VIN; no longer IC1.VI, IC2.VI, IC3.VI
- net N$10: now also IC1A.OUT, R8.2; no longer C14.1, IC5.VCC, L4.2, R2.2, R5.1, U$1.+3V3_A, U$1.+3V3_B
- net N$27: now also IC1C.OUT, R15.2; no longer C19.1, C20.1, IC4.VCC@1, IC4.VCC@2, L7.2, R6.1, SV1.2
- net N$28: now also IC1C.-IN, R17.2, R18.2; no longer C15.1, L2.2, R1.2, U$1.+12V_A, U$1.+12V_B
- net N$3: now also U$4.VOUT; no longer IC3.VO
- net N$4: now also U$3.VOUT; no longer D5.C, IC2.VO
- net N$5: now also U$2.VOUT; no longer IC1.VO
- net N$6: now also IC4.PC1(ADC1/PCINT9), U$1.SLOWCLK/CS; no longer C9.1, L5.2, L6.1
- net N$7: now also IC1A.-IN, R10.2, R9.2; no longer C4.1, L3.2, L4.1
- net N$8: now also IC1A.+IN, R7.2, R8.1; no longer C3.1, L1.2, L2.1
Other:
- note removed: "+12V"
- note removed: "+3.3V"
- note removed: "+5V"
- moved on the sheet: C1, C10, C11, C12, C13, C14, C15, C17, C18, C19, C2, C20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

Commit message: improved layout
Parts:
- removed LED1: (no value), led:LED3MM
- added JP2, JP3, JP4: (no value), pinhead:PINHD-1X1
- added LED3: GM5BW96385A, led:GM5BW96385A
- C15: value (none) -> 100n
- L1, L3, L5: value (none) -> 33u
- Q1: value (none) -> 20Mhz
- R1: value (none) -> 330
- R19, R20, R21: value (none) -> 0.01
- R2: value (none) -> 500
- R3: value (none) -> 1k2
- R4: value (none) -> 230
Connections:
- removed net N$10: IC1A.OUT, R8.2
- removed net N$11: IC1B.OUT, R13.2
- removed net N$27: IC1C.OUT, R15.2
- new net MEASURE12V: IC1C.OUT, IC4.PC5(ADC5/SCL/PCINT13), R15.2
- new net MEASURE3V3: IC1A.OUT, IC4.ADC6, R8.2
- new net MEASURE5V: IC1B.OUT, IC4.ADC7, R13.2
- net GND: now also JP4.1
- net N$19: now also LED3.C; no longer LED1.C
- net N$21: now also JP3.1
- net N$30: now also JP2.1
- net N$9: now also LED3.A; no longer LED1.A
- net TEMP1: now also IC4.PC0(ADC0/PCINT8); no longer IC4.ADC6

Commit message: less thrughhole parts
Parts:
- R1: device rcl:R-EU_0207/15 -> rcl:R-EU_R0805
- R2, R3: device rcl:R-EU_0207/15 -> rcl:R-EU_R0603
Changed lines of the file:
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@@
 <grid distance="0.1" unitdist="inch" unit="inch" style="lines" multiple="1" display="no" altdistance="0.01" altunitdist="inch" altunit="inch"/>
 <layers>
-<layer number="1" name="Top" color="4" fill="1" visible="no" active="no"/>
-<layer number="16" name="Bottom" color="1" fill="1" visible="no" active="no"/>
-<layer number="17" name="Pads" color="2" fill="1" visible="no" active="no"/>
-<layer number="18" name="Vias" color="2" fill="1" visible="no" active="no"/>
-<layer number="19" name="Unrouted" color="6" fill="1" visible="no" active="no"/>
-<layer number="20" name="Dimension" color="15" fill="1" visible="no" active="no"/>
-<layer number="21" name="tPlace" color="7" fill="1" visible="no" active="no"/>
-<layer number="22" name="bPlace" color="7" fill="1" visible="no" active="no"/>
-<layer number="23" name="tOrigins" color="15" fill="1" visible="no" active="no"/>
-<layer number="24" name="bOrigins" color="15" fill="1" visible="no" active="no"/>
-<layer number="25" name="tNames" color="7" fill="1" visible="no" active="no"/>
-<layer number="26" name="bNames" color="7" fill="1" visible="no" active="no"/>
-<layer number="27" name="tValues" color="7" fill="1" visible="no" active="no"/>
-<layer number="28" name="bValues" color="7" fill="1" visible="no" active="no"/>
+<layer number="1" name="Top" color="4" fill="1" visible="yes" active="no"/>
+<layer number="16" name="Bottom" color="1" fill="1" visible="yes" active="no"/>
+<layer number="17" name="Pads" color="2" fill="1" visible="yes" active="no"/>
+<layer number="18" name="Vias" color="2" fill="1" visible="yes" active="no"/>
+<layer number="19" name="Unrouted" color="6" fill="1" visible="yes" active="no"/>
+<layer number="20" name="Dimension" color="15" fill="1" visible="yes" active="no"/>
+<layer number="21" name="tPlace" color="7" fill="1" visible="yes" active="no"/>
+<layer number="22" name="bPlace" color="7" fill="1" visible="yes" active="no"/>
+<layer number="23" name="tOrigins" color="15" fill="1" visible="yes" active="no"/>
+<layer number="24" name="bOrigins" color="15" fill="1" visible="yes" active="no"/>
+<layer number="25" name="tNames" color="7" fill="1" visible="yes" active="no"/>
+<layer number="26" name="bNames" color="7" fill="1" visible="yes" active="no"/>
+<layer number="27" name="tValues" color="7" fill="1" visible="yes" active="no"/>
+<layer number="28" name="bValues" color="7" fill="1" visible="yes" active="no"/>
 <layer number="29" name="tStop" color="7" fill="3" visible="no" active="no"/>
 <layer number="30" name="bStop" color="7" fill="6" visible="no" active="no"/>
@@
 <layer number="35" name="tGlue" color="7" fill="4" visible="no" active="no"/>
 <layer number="36" name="bGlue" color="7" fill="5" visible="no" active="no"/>
-<layer number="37" name="tTest" color="7" fill="1" visible="no" active="no"/>
-<layer number="38" name="bTest" color="7" fill="1" visible="no" active="no"/>
+<layer number="37" name="tTest" color="7" fill="1" visible="yes" active="no"/>
+<layer number="38" name="bTest" color="7" fill="1" visible="yes" active="no"/>
 <layer number="39" name="tKeepout" color="4" fill="11" visible="no" active="no"/>
 <layer number="40" name="bKeepout" color="1" fill="11" visible="no" active="no"/>
@@
 <layer number="44" name="Drills" color="7" fill="1" visible="no" active="no"/>
 <layer number="45" name="Holes" color="7" fill="1" visible="no" active="no"/>
-<layer number="46" name="Milling" color="3" fill="1" visible="no" active="no"/>
-<layer number="47" name="Measures" color="7" fill="1" visible="no" active="no"/>
-<layer number="48" name="Document" color="7" fill="1" visible="no" active="no"/>
-<layer number="49" name="Reference" color="7" fill="1" visible="no" active="no"/>
-<layer number="50" name="dxf" color="7" fill="1" visible="no" active="no"/>
-<layer number="51" name="tDocu" color="7" fill="1" visible="no" active="no"/>
-<layer number="52" name="bDocu" color="7" fill="1" visible="no" active="no"/>
+<layer number="46" name="Milling" color="3" fill="1" visible="yes" active="no"/>
+<layer number="47" name="Measures" color="7" fill="1" visible="yes" active="no"/>
+<layer number="48" name="Document" color="7" fill="1" visible="yes" active="no"/>
+<layer number="49" name="Reference" color="7" fill="1" visible="yes" active="no"/>
+<layer number="50" name="dxf" color="7" fill="1" visible="yes" active="no"/>
+<layer number="51" name="tDocu" color="7" fill="1" visible="yes" active="no"/>
+<layer number="52" name="bDocu" color="7" fill="1" visible="yes" active="no"/>
 <layer number="91" name="Nets" color="2" fill="1" visible="yes" active="yes"/>
 <layer number="92" name="Busses" color="1" fill="1" visible="yes" active="yes"/>
@@
 <part name="GND20" library="supply1" deviceset="GND" device=""/>
 <part name="GND21" library="supply1" deviceset="GND" device=""/>
-<part name="R1" library="rcl" deviceset="R-EU_" device="0207/15" value="330"/>
-<part name="R2" library="rcl" deviceset="R-EU_" device="0207/15" value="500"/>
-<part name="R3" library="rcl" deviceset="R-EU_" device="0207/15" value="1k2"/>
+<part name="R1" library="rcl" deviceset="R-EU_" device="R0805" value="330"/>
+<part name="R2" library="rcl" deviceset="R-EU_" device="R0603" value="500"/>
+<part name="R3" library="rcl" deviceset="R-EU_" device="R0603" value="1k2"/>
 <part name="D1" library="diode" deviceset="1N4004" device=""/>
 <part name="D2" library="diode" deviceset="1N4004" device=""/>

Commit message: .
Parts:
- C13: device resistor:C-EU025-060X050 -> resistor:C-EU050-055X075
Changed lines of the file:
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@@
 <part name="L3" library="resistor" deviceset="L-EU" device="0207/5V" value="33u"/>
 <part name="L5" library="resistor" deviceset="L-EU" device="0207/5V" value="33u"/>
-<part name="C13" library="resistor" deviceset="C-EU" device="025-060X050" value="2000u"/>
+<part name="C13" library="resistor" deviceset="C-EU" device="050-055X075" value="2000u"/>
 <part name="GND18" library="supply1" deviceset="GND" device=""/>
 <part name="GND19" library="supply1" deviceset="GND" device=""/>

Commit message: updates versoin of braeburn
Parts:
- removed C11, C12: (no value), rcl:C-EU025-050X050
- removed C13: 2000u, resistor:C-EU050-055X075
- added C16, C21, C22: (no value), rcl:CPOL-EU153CLV-0505
- C10: device rcl:C-EU025-050X050 -> rcl:CPOL-EU150CLZ-1010
- Q1: device crystal:CRYSTALHC49U-V -> crystal:CRYSTALHC49UP; OC_FARNELL (none) -> unknown
Connections:
- removed net N$1: C1.1, C6.1, C7.1, D1.C, D2.C, D3.C, D4.C, U$2.VIN, U$3.VIN, U$4.VIN
- removed net N$3: C12.1, C8.1, D4.A, L5.1, U$4.VOUT
- removed net N$4: C11.1, C5.1, D2.A, L3.1, U$3.VOUT
- new net 12VOUT: C22.+, C6.1, C8.1, D2.C, D4.A, L5.1, U$3.VIN, U$4.VOUT
- new net 5VOUT: C1.1, C21.+, C5.1, D2.A, D3.C, L3.1, U$2.VIN, U$3.VOUT
- new net N$11: C7.1, D1.C, D4.C, U$4.VIN
- net 3V3: no longer U$1.+3V3_B
- net GND: now also C10.-, C16.-, C21.-, C22.-; no longer C10.2, C11.2, C12.2, C13.2, U$1.GND1_A, U$1.GND2_A, U$1.GND3_A
- net N$12: now also C10.+; no longer C13.1
- net N$5: now also C16.+; no longer C10.1
- net VCC: no longer U$1.+5V_B
Other:
- moved on the sheet: D1, X1-1, X1-2
